File: hardware/maxwell/power.sch (KiCad schematic (older format))
At the start: 35 parts, among them J7 Dynamo Input, J8 USB Input, J9 Battery, Q2 Q_NMOS_GDS, Q3 Q_PMOS_GDS, U10 LT1529, U8 TLP188, U9 Buck Regulator

Commit message: Continuing onward.
Parts:
- C15, C17, C19: symbol CP -> maxwell-rescue:CP-RESCUE-maxwell
- C16, C18, C20: symbol C -> maxwell-rescue:C-RESCUE-maxwell
- D1, D5, D6: symbol D -> maxwell-rescue:D-RESCUE-maxwell
- D2, D3: symbol D_Zener -> maxwell-rescue:D_Zener-RESCUE-maxwell
- D4: symbol D_Bridge_+-AA -> maxwell-rescue:D_Bridge_+-AA-RESCUE-maxwell
- J7, J9: symbol Conn_01x02 -> maxwell-rescue:Conn_01x02-RESCUE-maxwell
- J8: symbol USB_OTG -> maxwell-rescue:USB_OTG-RESCUE-maxwell
- Q2: symbol Q_NMOS_GDS -> maxwell-rescue:Q_NMOS_GDS-RESCUE-maxwell
- Q3: symbol Q_PMOS_GDS -> maxwell-rescue:Q_PMOS_GDS-RESCUE-maxwell
- R14, R15, R18, R19, R20, R21, R22, R23, R24, R25, R30, R34, R35, R36: symbol R -> maxwell-rescue:R-RESCUE-maxwell
- U*1: symbol MCP73831T -> maxwell-rescue:MCP73831T-RESCUE-maxwell
- U10: symbol LT1529 -> maxwell-rescue:LT1529-RESCUE-maxwell
- U8: symbol TLP185(SE -> maxwell-rescue:TLP185(SE-RESCUE-maxwell
- U9: symbol BOOST_BOARD -> maxwell-rescue:BOOST_BOARD-RESCUE-maxwell
Changed lines of the file:
@@
-EESchema Schematic File Version 3
-LIBS:power
-LIBS:device
-LIBS:transistors
-LIBS:conn
-LIBS:linear
-LIBS:regul
-LIBS:74xx
-LIBS:cmos4000
-LIBS:adc-dac
-LIBS:memory
-LIBS:xilinx
-LIBS:microcontrollers
-LIBS:dsp
-LIBS:microchip
-LIBS:analog_switches
-LIBS:motorola
-LIBS:texas
-LIBS:intel
-LIBS:audio
-LIBS:interface
-LIBS:digital-audio
-LIBS:philips
-LIBS:display
-LIBS:cypress
-LIBS:siliconi
-LIBS:opto
-LIBS:atmel
-LIBS:contrib
-LIBS:valves
-LIBS:stm32
-LIBS:coddingtonbear
-LIBS:mcp73831t
-LIBS:custom
-LIBS:w_rtx
+EESchema Schematic File Version 4
 LIBS:maxwell-cache
 EELAYER 26 0
@@
 $EndDescr
 $Comp
-L Conn_01x02 J7
+L maxwell-rescue:Conn_01x02-RESCUE-maxwell J7
 U 1 1 5A1FF249
 P 1500 1100
@@
 $EndComp
 $Comp
-L TLP185(SE U8
+L maxwell-rescue:TLP185(SE-RESCUE-maxwell U8
 U 1 1 5A1FF25C
 P 1800 2700
@@
 $EndComp
 $Comp
-L D D1
+L maxwell-rescue:D-RESCUE-maxwell D1
 U 1 1 5A1FF263
 P 1500 3250
@@
 $EndComp
 $Comp
-L R R15
+L maxwell-rescue:R-RESCUE-maxwell R15
 U 1 1 5A1FF270
 P 2100 2950
@@
 $EndComp
 $Comp
-L +3V3 #PWR032
+L maxwell-rescue:+3V3-RESCUE-maxwell #PWR032
 U 1 1 5A1FF277
 P 2100 2600
@@
 SPEED
 $Comp
-L D_Bridge_+-AA D4
+L maxwell-rescue:D_Bridge_+-AA-RESCUE-maxwell D4
 U 1 1 5A1FF27E
 P 3350 1250
@@
 $EndComp
 $Comp
-L GND #PWR033
+L maxwell-rescue:GND-RESCUE-maxwell #PWR033
 U 1 1 5A1FF28B
 P 3050 1250
@@
 $EndComp
 $Comp
-L R R14
+L maxwell-rescue:R-RESCUE-maxwell R14
 U 1 1 5A1FF297
 P 1500 2950
@@
 $EndComp
 $Comp
-L D_Zener D2
+L maxwell-rescue:D_Zener-RESCUE-maxwell D2
 U 1 1 5A1FF2A4
 P 2400 1050
@@
 $EndComp
 $Comp
-L D_Zener D3
+L maxwell-rescue:D_Zener-RESCUE-maxwell D3
 U 1 1 5A1FF2AB
 P 2400 1400
@@
 $EndComp
 $Comp
-L +3V3 #PWR035
+L maxwell-rescue:+3V3-RESCUE-maxwell #PWR035
 U 1 1 5A1FFDA9
 P 8200 3100
@@
 $EndComp
 $Comp
-L GND #PWR036
+L maxwell-rescue:GND-RESCUE-maxwell #PWR036
 U 1 1 5A1FFDAF
 P 7100 3500
@@
 $EndComp
 $Comp
-L USB_OTG J8
+L maxwell-rescue:USB_OTG-RESCUE-maxwell J8
 U 1 1 5A1FFDB5
 P 3400 2550
@@
 $EndComp
 $Comp
-L GND #PWR037
+L maxwell-rescue:GND-RESCUE-maxwell #PWR037
 U 1 1 5A1FFDBC
 P 3400 2950
@@
 USB+
 $Comp
-L C C20
+L maxwell-rescue:C-RESCUE-maxwell C20
 U 1 1 5A1FFDC5
 P 7850 3250
@@
 $EndComp
 $Comp
-L C C16
+L maxwell-rescue:C-RESCUE-maxwell C16
 U 1 1 5A1FFDCC
 P 5450 3250
@@
 $EndComp
 $Comp
-L CP C19
+L maxwell-rescue:CP-RESCUE-maxwell C19
 U 1 1 5A1FFDD3
 P 7500 3250
@@
 $EndComp
 $Comp
-L BOOST_BOARD U9
+L maxwell-rescue:BOOST_BOARD-RESCUE-maxwell U9
 U 1 1 5A1FFDEF
 P 4700 1300
@@
 $EndComp
 $Comp
-L GND #PWR038
+L maxwell-rescue:GND-RESCUE-maxwell #PWR038
 U 1 1 5A1FFDF6
 P 4200 1350
@@
 $EndComp
 $Comp
-L GND #PWR039
+L maxwell-rescue:GND-RESCUE-maxwell #PWR039
 U 1 1 5A1FFDFC
 P 5150 1350
@@
 $EndComp
 $Comp
-L CP C15
+L maxwell-rescue:CP-RESCUE-maxwell C15
 U 1 1 5A20260D
 P 3650 1600
@@
 $EndComp
 $Comp
-L GND #PWR040
+L maxwell-rescue:GND-RESCUE-maxwell #PWR040
 U 1 1 5A202661
 P 3650 1750
@@
 $EndComp
 $Comp
-L D D5
+L maxwell-rescue:D-RESCUE-maxwell D5
 U 1 1 5A202C41
 P 4100 2350
@@
 $EndComp
 $Comp
-L LT1529 U10
+L maxwell-rescue:LT1529-RESCUE-maxwell U10
 U 1 1 5A20F6E0
 P 7050 3200
@@
 $EndComp
 $Comp
-L MCP73831T U*1
+L maxwell-rescue:MCP73831T-RESCUE-maxwell U*1
 U 1 1 5A2102FA
 P 6850 1600
@@
 $EndComp
 $Comp
-L Conn_01x02 J9
+L maxwell-rescue:Conn_01x02-RESCUE-maxwell J9
 U 1 1 5A21040E
 P 8600 1250
@@
 $EndComp
 $Comp
-L GND #PWR041
+L maxwell-rescue:GND-RESCUE-maxwell #PWR041
 U 1 1 5A21058A
 P 7350 1900
@@
 $EndComp
 $Comp
-L GND #PWR042
+L maxwell-rescue:GND-RESCUE-maxwell #PWR042
 U 1 1 5A210626
 P 8400 1350
@@
 $EndComp
 $Comp
-L R R19
+L maxwell-rescue:R-RESCUE-maxwell R19
 U 1 1 5A210718
 P 7450 1650
@@
 Tune to 4V
 $Comp
-L +BATT #PWR044
+L maxwell-rescue:+BATT-RESCUE-maxwell #PWR044
 U 1 1 5A2124F4
 P 5450 3000
@@
 $EndComp
 $Comp
-L C C18
+L maxwell-rescue:C-RESCUE-maxwell C18
 U 1 1 5A22422F
 P 5900 1450
@@
 $EndComp
 $Comp
-L GND #PWR045
+L maxwell-rescue:GND-RESCUE-maxwell #PWR045
 U 1 1 5A2243E8
 P 5900 2050
@@
 $EndComp
 $Comp
-L R R18
+L maxwell-rescue:R-RESCUE-maxwell R18
 U 1 1 5A2253E0
 P 6350 3200
@@
 µC should hold\nPOWER_ON high\nupon startup
 $Comp
-L D D6
+L maxwell-rescue:D-RESCUE-maxwell D6
 U 1 1 5A226F08
 P 6200 4150
@@
 $EndComp
 $Comp
-L R R20
+L maxwell-rescue:R-RESCUE-maxwell R20
 U 1 1 5A245A23
 P 9300 1250
@@
 $EndComp
 $Comp
-L R R21
+L maxwell-rescue:R-RESCUE-maxwell R21
 U 1 1 5A245A89
 P 9300 1650
@@
 $EndComp
 $Comp
-L R R23
+L maxwell-rescue:R-RESCUE-maxwell R23
 U 1 1 5A245B4A
 P 10100 1250
@@
 $EndComp
 $Comp
-L R R24
+L maxwell-rescue:R-RESCUE-maxwell R24
 U 1 1 5A245B93
 P 10100 1650
@@
 $EndComp
 $Comp
-L R R22
+L maxwell-rescue:R-RESCUE-maxwell R22
 U 1 1 5A246038
 P 9700 1100
@@
 BATT_VOLTAGE
 $Comp
-L CP C17
+L maxwell-rescue:CP-RESCUE-maxwell C17
 U 1 1 5A24B0B8
 P 5650 1450
@@
 $EndComp
 $Comp
-L Q_NMOS_GDS Q2
+L maxwell-rescue:Q_NMOS_GDS-RESCUE-maxwell Q2
 U 1 1 5A257F55
 P 3150 3900
@@
 $EndComp
 $Comp
-L GNDPWR #PWR049
+L maxwell-rescue:GNDPWR-RESCUE-maxwell #PWR049
 U 1 1 5A25809F
 P 3500 3700
@@
 $EndComp
 $Comp
-L GND #PWR050
+L maxwell-rescue:GND-RESCUE-maxwell #PWR050
 U 1 1 5A2580F1
 P 3250 4200
@@
 $EndComp
 $Comp
-L R R25
+L maxwell-rescue:R-RESCUE-maxwell R25
 U 1 1 5A25869F
 P 2850 4150
@@
 DYNAMO_NEUTRAL
 $Comp
-L R R30
+L maxwell-rescue:R-RESCUE-maxwell R30
 U 1 1 5A26A72F
 P 6650 2500
@@
 ~BATT_CHARGE_ENABLE
 $Comp
-L R R34
+L maxwell-rescue:R-RESCUE-maxwell R34
 U 1 1 5A27817C
 P 4150 850
@@
 $EndComp
 $Comp
-L R R35
+L maxwell-rescue:R-RESCUE-maxwell R35
 U 1 1 5A2781E1
 P 4500 850
@@
 $EndComp
 $Comp
-L GND #PWR046
+L maxwell-rescue:GND-RESCUE-maxwell #PWR046
 U 1 1 5A278243
 P 4650 850
@@
 DYNAMO_VOLTAGE
 $Comp
-L R R36
+L maxwell-rescue:R-RESCUE-maxwell R36
 U 1 1 5A27BDA2
 P 5350 750
@@
 $EndComp
 $Comp
-L +BATT #PWR043
+L maxwell-rescue:+BATT-RESCUE-maxwell #PWR043
 U 1 1 5A210C7A
 P 10250 1100
@@
 Connection ~ 5400 950
 $Comp
-L Q_PMOS_GDS Q3
+L maxwell-rescue:Q_PMOS_GDS-RESCUE-maxwell Q3
 U 1 1 5A2B17F5
 P 5400 1150
@@
 	5450 3000 5450 3100
 $Comp
-L GNDPWR #PWR020
+L maxwell-rescue:GNDPWR-RESCUE-maxwell #PWR020
 U 1 1 5A2C7A67
 P 9300 1950
