File: hardware/maxwell/maxwell.sch (KiCad schematic (older format))
At the start: 31 parts, among them J1 Canbus 1, J10 SPI2_B, J11 BACKUP, J12 UART4, J13 UART5, J14 I2C1, J16 ESP_BM, J17 ESP_PROG, J2 Canbus 2, J3 Neopixel, J4 BOOT0, J5 SPI2_A, J6 Programmer, J8 BOOT1, Q1 BSS138, U2 SN65HVD233, U5 ESP-32S

Commit message: Updating hardware to reference the proper libraries; adding new parts to board to support switching from dynamo input to battery.
Parts:
- BZ1: footprint coddingtonbear/coddingtonbear.pretty:12mm_buzzer -> coddingtonbear:12mm_buzzer
- C4, C5, R1, R16, R2, R31, R37, R4, R5, R6, R7, R8, R9: footprint coddingtonbear/coddingtonbear.pretty:0805_Milling -> coddingtonbear:0805_Milling
- J1, J2: footprint coddingtonbear/coddingtonbear.pretty:JST_XH_B05B-XH-A_05x2.50mm_Straight_LargePads -> coddingtonbear:JST_XH_B05B-XH-A_05x2.50mm_Straight_LargePads
- J10, J5: footprint coddingtonbear/coddingtonbear.pretty:JST_XH_B06B-XH-A_06x2.50mm_Straight_LargePads -> coddingtonbear:JST_XH_B06B-XH-A_06x2.50mm_Straight_LargePads
- J11: footprint coddingtonbear/coddingtonbear.pretty:JST_XH_B02B-XH-A_02x2.50mm_Straight_LargePads -> coddingtonbear:JST_XH_B02B-XH-A_02x2.50mm_Straight_LargePads
- J12, J13, J14: footprint coddingtonbear/coddingtonbear.pretty:JST_XH_B04B-XH-A_04x2.50mm_Straight_LargePads -> coddingtonbear:JST_XH_B04B-XH-A_04x2.50mm_Straight_LargePads
- J16: footprint coddingtonbear/coddingtonbear.pretty:Pin_Header_Straight_1x02_Pitch1.27mm_JMP -> coddingtonbear:Pin_Header_Straight_1x02_Pitch1.27mm_JMP
- J17, J3: footprint coddingtonbear/coddingtonbear.pretty:JST_XH_B03B-XH-A_03x2.50mm_Straight_LargePads -> coddingtonbear:JST_XH_B03B-XH-A_03x2.50mm_Straight_LargePads
- J6: footprint KiCad/Pin_Headers.pretty:Pin_Header_Straight_1x04_Pitch2.54mm -> coddingtonbear:Pin_Header_Straight_1x04_Pitch2.54mm_LargePads
- Q1: footprint coddingtonbear/coddingtonbear.pretty:SOT-23_LargePads -> coddingtonbear:SOT-23_LargePads
- U2: footprint adamgreig/agg-kicad/agg.pretty:SOIC-8 -> coddingtonbear:SOIC-8_3.9x4.9mm_P1.27mm_LargePads
- U5: footprint coddingtonbear/coddingtonbear.pretty:ESP-32S -> coddingtonbear:ESP-32S
Changed lines of the file:
@@
 F 0 "J6" H 2430 3392 50  0000 L CNN
 F 1 "Programmer" H 2430 3301 50  0000 L CNN
-F 2 "KiCad/Pin_Headers.pretty:Pin_Header_Straight_1x04_Pitch2.54mm" H 2350 3400 50  0001 C CNN
+F 2 "coddingtonbear:Pin_Header_Straight_1x04_Pitch2.54mm_LargePads" H 2350 3400 50  0001 C CNN
 F 3 "" H 2350 3400 50  0001 C CNN
 	1    2350 3400
@@
 F 0 "R8" V 1193 3600 50  0000 C CNN
 F 1 "10k" V 1284 3600 50  0000 C CNN
-F 2 "coddingtonbear/coddingtonbear.pretty:0805_Milling" V 1330 3600 50  0001 C CNN
+F 2 "coddingtonbear:0805_Milling" V 1330 3600 50  0001 C CNN
 F 3 "" H 1400 3600 50  0001 C CNN
 	1    1400 3600
@@
 F 0 "R7" V 1193 3300 50  0000 C CNN
 F 1 "10k" V 1284 3300 50  0000 C CNN
-F 2 "coddingtonbear/coddingtonbear.pretty:0805_Milling" V 1330 3300 50  0001 C CNN
+F 2 "coddingtonbear:0805_Milling" V 1330 3300 50  0001 C CNN
 F 3 "" H 1400 3300 50  0001 C CNN
 	1    1400 3300
@@
 F 0 "U2" H 1550 6428 50  0000 C CNN
 F 1 "SN65HVD233" H 1550 6337 50  0000 C CNN
-F 2 "adamgreig/agg-kicad/agg.pretty:SOIC-8" H 1550 5450 50  0001 C CNN
+F 2 "coddingtonbear:SOIC-8_3.9x4.9mm_P1.27mm_LargePads" H 1550 5450 50  0001 C CNN
 F 3 "" H 1450 6350 50  0001 C CNN
 	1    1550 5950
@@
 F 0 "R1" H 1070 6346 50  0000 L CNN
 F 1 "10k" H 1070 6255 50  0000 L CNN
-F 2 "coddingtonbear/coddingtonbear.pretty:0805_Milling" V 930 6300 50  0001 C CNN
+F 2 "coddingtonbear:0805_Milling" V 930 6300 50  0001 C CNN
 F 3 "" H 1000 6300 50  0001 C CNN
 	1    1000 6300
@@
 F 0 "C4" V 1448 5350 50  0000 C CNN
 F 1 "0.1u" V 1539 5350 50  0000 C CNN
-F 2 "coddingtonbear/coddingtonbear.pretty:0805_Milling" H 1738 5200 50  0001 C CNN
+F 2 "coddingtonbear:0805_Milling" H 1738 5200 50  0001 C CNN
 F 3 "" H 1700 5350 50  0001 C CNN
 	1    1700 5350
@@
 F 0 "BZ1" H 4153 3929 50  0000 L CNN
 F 1 "Buzzer" H 4153 3838 50  0000 L CNN
-F 2 "coddingtonbear/coddingtonbear.pretty:12mm_buzzer" V 3975 4000 50  0001 C CNN
+F 2 "coddingtonbear:12mm_buzzer" V 3975 4000 50  0001 C CNN
 F 3 "" V 3975 4000 50  0001 C CNN
 	1    4000 3900
@@
 F 0 "Q1" V 4143 4200 50  0000 C CNN
 F 1 "BSS138" V 4052 4200 50  0000 C CNN
-F 2 "coddingtonbear/coddingtonbear.pretty:SOT-23_LargePads" H 4000 4125 50  0001 L CIN
+F 2 "coddingtonbear:SOT-23_LargePads" H 4000 4125 50  0001 L CIN
 F 3 "" H 3800 4200 50  0001 L CNN
 	1    3800 4200
@@
 F 0 "J3" H 2230 4592 50  0000 L CNN
 F 1 "Neopixel" H 2230 4501 50  0000 L CNN
-F 2 "coddingtonbear/coddingtonbear.pretty:JST_XH_B03B-XH-A_03x2.50mm_Straight_LargePads" H 2150 4550 50  0001 C CNN
+F 2 "coddingtonbear:JST_XH_B03B-XH-A_03x2.50mm_Straight_LargePads" H 2150 4550 50  0001 C CNN
 F 3 "" H 2150 4550 50  0001 C CNN
 	1    2150 4550
@@
 F 0 "J1" H 2830 5992 50  0000 L CNN
 F 1 "Canbus 1" H 2830 5901 50  0000 L CNN
-F 2 "coddingtonbear/coddingtonbear.pretty:JST_XH_B05B-XH-A_05x2.50mm_Straight_LargePads" H 2750 5950 50  0001 C CNN
+F 2 "coddingtonbear:JST_XH_B05B-XH-A_05x2.50mm_Straight_LargePads" H 2750 5950 50  0001 C CNN
 F 3 "" H 2750 5950 50  0001 C CNN
 	1    2750 5950
@@
 F 0 "J2" H 2830 6592 50  0000 L CNN
 F 1 "Canbus 2" H 2830 6501 50  0000 L CNN
-F 2 "coddingtonbear/coddingtonbear.pretty:JST_XH_B05B-XH-A_05x2.50mm_Straight_LargePads" H 2750 6550 50  0001 C CNN
+F 2 "coddingtonbear:JST_XH_B05B-XH-A_05x2.50mm_Straight_LargePads" H 2750 6550 50  0001 C CNN
 F 3 "" H 2750 6550 50  0001 C CNN
 	1    2750 6550
@@
 F 0 "R31" H 1670 4596 50  0000 L CNN
 F 1 "330" H 1670 4505 50  0000 L CNN
-F 2 "coddingtonbear/coddingtonbear.pretty:0805_Milling" V 1530 4550 50  0001 C CNN
+F 2 "coddingtonbear:0805_Milling" V 1530 4550 50  0001 C CNN
 F 3 "" H 1600 4550 50  0001 C CNN
 	1    1600 4550
@@
 F 0 "R4" V 3693 4600 50  0000 C CNN
 F 1 ">35" V 3784 4600 50  0000 C CNN
-F 2 "coddingtonbear/coddingtonbear.pretty:0805_Milling" V 3830 4600 50  0001 C CNN
+F 2 "coddingtonbear:0805_Milling" V 3830 4600 50  0001 C CNN
 F 3 "" H 3900 4600 50  0001 C CNN
 	1    3900 4600
@@
 F 0 "R37" H 2070 6646 50  0000 L CNN
 F 1 "120" H 2070 6555 50  0000 L CNN
-F 2 "coddingtonbear/coddingtonbear.pretty:0805_Milling" V 1930 6600 50  0001 C CNN
+F 2 "coddingtonbear:0805_Milling" V 1930 6600 50  0001 C CNN
 F 3 "" H 2000 6600 50  0001 C CNN
 	1    2000 6600
@@
 F 0 "R5" H 3120 1446 50  0000 L CNN
 F 1 "100k" H 3120 1355 50  0000 L CNN
-F 2 "coddingtonbear/coddingtonbear.pretty:0805_Milling" V 2980 1400 50  0001 C CNN
+F 2 "coddingtonbear:0805_Milling" V 2980 1400 50  0001 C CNN
 F 3 "" H 3050 1400 50  0001 C CNN
 	1    3050 1400
@@
 F 0 "R9" H 3120 2696 50  0000 L CNN
 F 1 "100k" H 3120 2605 50  0000 L CNN
-F 2 "coddingtonbear/coddingtonbear.pretty:0805_Milling" V 2980 2650 50  0001 C CNN
+F 2 "coddingtonbear:0805_Milling" V 2980 2650 50  0001 C CNN
 F 3 "" H 3050 2650 50  0001 C CNN
 	1    3050 2650
@@
 F 0 "J5" H 8029 1542 50  0000 L CNN
 F 1 "SPI2_A" H 8029 1451 50  0000 L CNN
-F 2 "coddingtonbear/coddingtonbear.pretty:JST_XH_B06B-XH-A_06x2.50mm_Straight_LargePads" H 7950 1550 50  0001 C CNN
+F 2 "coddingtonbear:JST_XH_B06B-XH-A_06x2.50mm_Straight_LargePads" H 7950 1550 50  0001 C CNN
 F 3 "~" H 7950 1550 50  0001 C CNN
 	1    7950 1550
@@
 F 0 "J10" H 8430 1542 50  0000 L CNN
 F 1 "SPI2_B" H 8430 1451 50  0000 L CNN
-F 2 "coddingtonbear/coddingtonbear.pretty:JST_XH_B06B-XH-A_06x2.50mm_Straight_LargePads" H 8350 1550 50  0001 C CNN
+F 2 "coddingtonbear:JST_XH_B06B-XH-A_06x2.50mm_Straight_LargePads" H 8350 1550 50  0001 C CNN
 F 3 "~" H 8350 1550 50  0001 C CNN
 	1    8350 1550
@@
 F 0 "U5" V 9322 4728 60  0000 L CNN
 F 1 "ESP-32S" V 9428 4728 60  0000 L CNN
-F 2 "coddingtonbear/coddingtonbear.pretty:ESP-32S" H 9750 4850 60  0001 C CNN
+F 2 "coddingtonbear:ESP-32S" H 9750 4850 60  0001 C CNN
 F 3 "" H 8950 3950 60  0001 C CNN
 	1    9400 3500
@@
 F 0 "R6" H 8120 3046 50  0000 L CNN
 F 1 "10k" H 8120 2955 50  0000 L CNN
-F 2 "coddingtonbear/coddingtonbear.pretty:0805_Milling" V 7980 3000 50  0001 C CNN
+F 2 "coddingtonbear:0805_Milling" V 7980 3000 50  0001 C CNN
 F 3 "" H 8050 3000 50  0001 C CNN
 	1    8050 3000
@@
 F 0 "J11" H 2630 2042 50  0000 L CNN
 F 1 "BACKUP" H 2630 1951 50  0000 L CNN
-F 2 "coddingtonbear/coddingtonbear.pretty:JST_XH_B02B-XH-A_02x2.50mm_Straight_LargePads" H 2550 2050 50  0001 C CNN
+F 2 "coddingtonbear:JST_XH_B02B-XH-A_02x2.50mm_Straight_LargePads" H 2550 2050 50  0001 C CNN
 F 3 "~" H 2550 2050 50  0001 C CNN
 	1    2550 2050
@@
 F 0 "J12" H 4530 5692 50  0000 L CNN
 F 1 "UART4" H 4530 5601 50  0000 L CNN
-F 2 "coddingtonbear/coddingtonbear.pretty:JST_XH_B04B-XH-A_04x2.50mm_Straight_LargePads" H 4450 5700 50  0001 C CNN
+F 2 "coddingtonbear:JST_XH_B04B-XH-A_04x2.50mm_Straight_LargePads" H 4450 5700 50  0001 C CNN
 F 3 "~" H 4450 5700 50  0001 C CNN
 	1    4450 5700
@@
 F 0 "J13" H 4530 6192 50  0000 L CNN
 F 1 "UART5" H 4530 6101 50  0000 L CNN
-F 2 "coddingtonbear/coddingtonbear.pretty:JST_XH_B04B-XH-A_04x2.50mm_Straight_LargePads" H 4450 6200 50  0001 C CNN
+F 2 "coddingtonbear:JST_XH_B04B-XH-A_04x2.50mm_Straight_LargePads" H 4450 6200 50  0001 C CNN
 F 3 "~" H 4450 6200 50  0001 C CNN
 	1    4450 6200
@@
 F 0 "J14" H 5880 5742 50  0000 L CNN
 F 1 "I2C1" H 5880 5651 50  0000 L CNN
-F 2 "coddingtonbear/coddingtonbear.pretty:JST_XH_B04B-XH-A_04x2.50mm_Straight_LargePads" H 5800 5750 50  0001 C CNN
+F 2 "coddingtonbear:JST_XH_B04B-XH-A_04x2.50mm_Straight_LargePads" H 5800 5750 50  0001 C CNN
 F 3 "~" H 5800 5750 50  0001 C CNN
 	1    5800 5750
@@
 F 0 "R2" V 5193 6150 50  0000 C CNN
 F 1 "2.2k" V 5284 6150 50  0000 C CNN
-F 2 "coddingtonbear/coddingtonbear.pretty:0805_Milling" V 5330 6150 50  0001 C CNN
+F 2 "coddingtonbear:0805_Milling" V 5330 6150 50  0001 C CNN
 F 3 "" H 5400 6150 50  0001 C CNN
 	1    5400 6150
@@
 F 0 "R16" V 5343 6150 50  0000 C CNN
 F 1 "2.2k" V 5434 6150 50  0000 C CNN
-F 2 "coddingtonbear/coddingtonbear.pretty:0805_Milling" V 5480 6150 50  0001 C CNN
+F 2 "coddingtonbear:0805_Milling" V 5480 6150 50  0001 C CNN
 F 3 "" H 5550 6150 50  0001 C CNN
 	1    5550 6150
@@
 F 0 "C5" H 8015 2796 50  0000 L CNN
 F 1 "0.1u" H 8015 2705 50  0000 L CNN
-F 2 "coddingtonbear/coddingtonbear.pretty:0805_Milling" H 7938 2600 50  0001 C CNN
+F 2 "coddingtonbear:0805_Milling" H 7938 2600 50  0001 C CNN
 F 3 "" H 7900 2750 50  0001 C CNN
 	1    7900 2750
@@
 F 0 "J16" H 5579 2092 50  0000 L CNN
 F 1 "ESP_BM" H 5579 2001 50  0000 L CNN
-F 2 "coddingtonbear/coddingtonbear.pretty:Pin_Header_Straight_1x02_Pitch1.27mm_JMP" H 5500 2100 50  0001 C CNN
+F 2 "coddingtonbear:Pin_Header_Straight_1x02_Pitch1.27mm_JMP" H 5500 2100 50  0001 C CNN
 F 3 "~" H 5500 2100 50  0001 C CNN
 	1    5500 2100
@@
 F 0 "J17" H 6680 2242 50  0000 L CNN
 F 1 "ESP_PROG" H 6680 2151 50  0000 L CNN
-F 2 "coddingtonbear/coddingtonbear.pretty:JST_XH_B03B-XH-A_03x2.50mm_Straight_LargePads" H 6600 2200 50  0001 C CNN
+F 2 "coddingtonbear:JST_XH_B03B-XH-A_03x2.50mm_Straight_LargePads" H 6600 2200 50  0001 C CNN
 F 3 "" H 6600 2200 50  0001 C CNN
 	1    6600 2200

Commit message: v1.5 ready for production.
Parts:
- removed J2: Canbus 2, coddingtonbear:JST_XH_B05B-XH-A_05x2.50mm_Straight_LargePads, symbol maxwell-rescue:Conn_01x05-RESCUE-maxwell
- added J19: Interconnect (Power), coddingtonbear:IDC-Header_2x08_P2.54mm_Vertical_Largepads, symbol Connector_Generic:Conn_02x08_Odd_Even
- added J2: SPI2_C, coddingtonbear:JST_XH_B06B-XH-A_06x2.50mm_Straight_LargePads, symbol maxwell-rescue:Conn_01x06-conn
- added J20: Interconnect (uC), coddingtonbear:IDC-Header_2x08_P2.54mm_Vertical_Largepads, symbol Connector_Generic:Conn_02x08_Odd_Even
Connections:
- net +3V3: now also J19.1 (Pin_1), J19.3 (Pin_3), J19.5 (Pin_5), J19.7 (Pin_7), J20.1 (Pin_1), J20.3 (Pin_3), J20.5 (Pin_5), J20.7 (Pin_7)
- net BT_DI: now also U5.13 (IO14); no longer U5.24 (IO2)
- net BT_DO: now also U5.12 (IO27); no longer U5.23 (IO15)
- net GND: now also J19.10 (Pin_10), J19.11 (Pin_11), J19.12 (Pin_12), J19.14 (Pin_14), J19.9 (Pin_9), J2.6 (Pin_6), J20.10 (Pin_10), J20.11 (Pin_11), J20.12 (Pin_12), J20.14 (Pin_14), J20.9 (Pin_9)
- net I2C1_SCL: now also J19.16 (Pin_16), J20.16 (Pin_16)
- net I2C1_SDA: now also J19.15 (Pin_15), J20.15 (Pin_15)
- net SPI2_MISO: now also J2.4 (Pin_4)
- net SPI2_MOSI: now also J2.5 (Pin_5)
- net SPI2_SCK: now also J2.3 (Pin_3)
- net VCC: now also J19.2 (Pin_2), J19.4 (Pin_4), J19.6 (Pin_6), J19.8 (Pin_8), J2.2 (Pin_2), J20.2 (Pin_2), J20.4 (Pin_4), J20.6 (Pin_6), J20.8 (Pin_8)
- new net SPEED: J19.13 (Pin_13), J20.13 (Pin_13)
- new net SPI2_CS_C: J2.1 (Pin_1)
Other:
- moved on the sheet: BZ1, J16, J17, Q1, R4
