File: hardware/maxwell/microcontroller.sch (KiCad schematic (older format))
At the start: 18 parts, among them U7 STM32F103RETx, Y2 8M, Y3 32.768k

Commit message: Updating schematic/layout to latest kicad version.
Changed lines of the file:
@@
 $EndComp
 Wire Wire Line
-	8500 3450 9000 3450
+	8500 3450 8900 3450
 Wire Wire Line
 	9400 3450 9300 3450
@@
 $EndComp
 Wire Wire Line
-	2150 3450 2150 3750
+	2150 3450 2150 3600
 Wire Wire Line
 	1950 3650 1950 3600
@@
 $EndComp
 Wire Wire Line
-	2150 5250 2150 5550
+	2150 5250 2150 5400
 Wire Wire Line
 	1950 5400 2150 5400
@@
 	5500 5850 5500 6050
 Wire Wire Line
-	5500 6050 5900 6050
+	5500 6050 5600 6050
 Wire Wire Line
 	5600 5850 5600 6050
@@
 $EndComp
 Wire Wire Line
-	2800 2250 2900 2250
+	2800 2250 2850 2250
 Wire Wire Line
 	2500 2250 2350 2250
@@
 $EndComp
 Wire Wire Line
-	5900 1650 5900 1850
-Wire Wire Line
-	5800 1650 5800 1850
-Wire Wire Line
-	5700 1650 5700 1850
-Wire Wire Line
-	5600 1650 5600 1850
-Wire Wire Line
-	5500 1650 5500 1850
-Wire Wire Line
-	5200 1750 5900 1750
+	5900 1650 5900 1750
+Wire Wire Line
+	5800 1650 5800 1750
+Wire Wire Line
+	5700 1650 5700 1750
+Wire Wire Line
+	5600 1650 5600 1750
+Wire Wire Line
+	5500 1650 5500 1750
+Wire Wire Line
+	5200 1750 5500 1750
 Connection ~ 5500 1750
 Connection ~ 5600 1750
@@
 Connection ~ 5900 1750
 Wire Wire Line
-	5500 1350 5900 1350
+	5500 1350 5600 1350
 Connection ~ 5800 1350
 Connection ~ 5700 1350
@@
 	2800 5550 2450 5550
 Wire Wire Line
-	2450 3450 2800 3450
+	2450 3450 2700 3450
 Wire Wire Line
 	2800 3450 2800 3550
@@
 Connection ~ 2700 3450
 Wire Wire Line
-	2450 3750 2800 3750
+	2450 3750 2700 3750
 Wire Wire Line
 	2800 3750 2800 3650
@@
 Text GLabel 8500 5350 2    60   Output ~ 0
 ~BATT_CHARGE_ENABLE
+Wire Wire Line
+	8900 3450 9000 3450
+Wire Wire Line
+	2150 3600 2150 3750
+Wire Wire Line
+	2150 5400 2150 5550
+Wire Wire Line
+	5600 6050 5700 6050
+Wire Wire Line
+	5700 6050 5800 6050
+Wire Wire Line
+	5800 6050 5900 6050
+Wire Wire Line
+	5500 1750 5500 1850
+Wire Wire Line
+	5500 1750 5600 1750
+Wire Wire Line
+	5600 1750 5600 1850
+Wire Wire Line
+	5600 1750 5700 1750
+Wire Wire Line
+	5700 1750 5700 1850
+Wire Wire Line
+	5700 1750 5800 1750
+Wire Wire Line
+	5800 1750 5800 1850
+Wire Wire Line
+	5800 1750 5900 1750
+Wire Wire Line
+	5900 1750 5900 1850
+Wire Wire Line
+	5800 1350 5900 1350
+Wire Wire Line
+	5700 1350 5800 1350
+Wire Wire Line
+	5600 1350 5700 1350
+Wire Wire Line
+	2850 2250 2900 2250
+Wire Wire Line
+	2700 3450 2800 3450
+Wire Wire Line
+	2700 3750 2800 3750
 $EndSCHEMATC

Commit message: Maxwell Board v2.0;
Adds:

* On-board P-MOS polarity protection.
* Adds On-board GPS (PA6C)
* Adds On-board WIFI, and BLE (ESP32)
* Connectors for 2x external UART devices.
* Connectors for 2x external SPI devices.
* Connector for I2C devices.

Removals:

* Removes on-board GSM; will add later via UART connectors mentioned
  above.
* Removes on-board boost charging.  Can later add this functionality via
  provided connectors.

Changes:

* Although the GNDPWR ground reference still exists, only neopixels
  are switched off via it.  The quiescent current of the GPS module
  and the ESP32 can be controlled via other means.
* Swaps many of the ICs used for switching and power regulation.
* Removes boot jumper bank.  I very rarely used it, and the HC-05
  has now been proven to work for switching boot modes for remote
  flashing.
* Removes natural powered-off state previously handled bydisabling the
  voltage regulator until POWER_ON was pulled high.  This will
  undoubtedly decrease how long the device will be able to operate due
  to increased quiescent currents, but I am willing to accept that given
  that removing that logic makes the design and software (especially
  around keeping the device on while flashing) simpler.
* Many other minor things.
Parts:
- removed C14: 100n, coddingtonbear/coddingtonbear.pretty:0805_Milling, symbol maxwell-rescue:C-RESCUE-maxwell
- removed R12: 1.5k, coddingtonbear/coddingtonbear.pretty:0805_Milling, symbol maxwell-rescue:R-RESCUE-maxwell
- removed R13: 20, coddingtonbear/coddingtonbear.pretty:0805_Milling, symbol maxwell-rescue:R-RESCUE-maxwell
- removed R26: 1k, coddingtonbear/coddingtonbear.pretty:0805_Milling, symbol maxwell-rescue:R-RESCUE-maxwell
- removed Y3: 32.768k, f4grx/f4libs_th.pretty:XTAL32K, symbol maxwell-rescue:Crystal-RESCUE-maxwell
- added C1, C2: 2.2u, coddingtonbear:CP_Tantalum_Case-C_EIA-6032-28_Milling, symbol device:CP
- added J15: GPIO, KiCad/Pin_Headers.pretty:Pin_Header_Straight_1x03_Pitch2.54mm, symbol conn:Conn_01x03
- added U1: MCP1501, adamgreig/agg-kicad/agg.pretty:SOT-23-6, symbol coddingtonbear:MCP1501
- added Y1: 32.768k, KiCad/Crystals.pretty:Crystal_SMD_SeikoEpson_MC306-4pin_8.0x3.2mm, symbol device:Crystal_GND23_Small
- R11: value 20 -> 50
- Y2: footprint SchrodingersGat/Components.pretty:crystal_hc-49s -> nqbit/NQBit.pretty:HC-49USX_SMD
Connections:
- net labels added: +BACKUP, BT_DI, BT_DO, CAN_RX, CAN_TX, ESP_BOOT_MODE, ESP_DI, ESP_DO, GPS_DI, GPS_DO, I2C1_SCL, I2C1_SDA, SPI2_CS_A, SPI2_CS_B, SPI2_MISO, SPI2_MOSI, SPI2_SCK, UART4_RX, UART4_TX, UART5_RX, UART5_TX, ~DISABLE_ESP
- net labels removed: CAN_INT, GSM_RST, GSM_RXD, GSM_TXD, MISO, MOSI, RXD, SCK, TXD, USB+, USB-, USB_PRER+, USB_PRER-, ~CAN_CS, ~ENABLE_USB_OUT
- wire segments 62 -> 83
- no-connect marks 0 -> 11
Other:
- note removed: "V=(100*INPUT+47*INPUT)/100"

Commit message: Updating for manufacture.
Parts:
- U7: footprint kicad-castellated-breakouts:QFP64-1.27MM-CASTELLATED -> kicad-castellated-breakouts:QFP64-1.27MM-CASTELLATED-VERS
- Y2: footprint nqbit/NQBit.pretty:HC-49USX_SMD -> cpavlina/kicad-pcblib/smd-non-ipc.pretty:Abracon-ABM2
Connections:
- net labels added: BATT_SOURCE_DISABLE, CAN_DISABLE
- net labels removed: DYNAMO_VOLTAGE, ESP_BOOT_MODE, ESP_DI, ESP_DO
- no-connect marks 11 -> 8
Changed lines of the file:
@@
 F 0 "U7" H 5700 6028 50  0000 C CNN
 F 1 "STM32F103RETx" H 5700 5937 50  0000 C CNN
-F 2 "kicad-castellated-breakouts:QFP64-1.27MM-CASTELLATED" H 8400 5725 50  0001 R TNN
+F 2 "kicad-castellated-breakouts:QFP64-1.27MM-CASTELLATED-VERS" H 8400 5725 50  0001 R TNN
 F 3 "" H 5700 3850 50  0001 C CNN
 	1    5700 3850
@@
 F 0 "Y2" V 2404 3731 50  0000 L CNN
 F 1 "8M" V 2495 3731 50  0000 L CNN
-F 2 "nqbit/NQBit.pretty:HC-49USX_SMD" H 2450 3600 50  0001 C CNN
+F 2 "cpavlina/kicad-pcblib/smd-non-ipc.pretty:Abracon-ABM2" H 2450 3600 50  0001 C CNN
 F 3 "" H 2450 3600 50  0001 C CNN
 	1    2450 3600
@@
 Text GLabel 8500 3250 2    60   Input ~ 0
 BT_DO
-Text GLabel 8500 3350 2    60   Output ~ 0
+Text GLabel 2900 4550 0    60   Output ~ 0
 BT_KEY
 Text GLabel 2900 4050 0    60   Input ~ 0
@@
 	2800 3650 2900 3650
 Connection ~ 2700 3750
-Text GLabel 2900 4250 0    60   Input ~ 0
-DYNAMO_VOLTAGE
+Text GLabel 2900 4250 0    60   Output ~ 0
+CAN_DISABLE
 Text GLabel 2000 5150 0    60   Output ~ 0
 ~BATT_CHARGE_ENABLE
@@
 Wire Wire Line
 	2550 5550 2450 5550
-Text GLabel 2900 4650 0    60   Output ~ 0
+Text GLabel 8500 2650 2    60   Output ~ 0
 SPI2_CS_A
-Text GLabel 8500 5250 2    60   Output ~ 0
+Text GLabel 8500 5450 2    60   Output ~ 0
 SPI2_MOSI
 Text GLabel 8500 5350 2    60   Input ~ 0
 SPI2_MISO
-Text GLabel 8500 5450 2    60   Output ~ 0
+Text GLabel 8500 5250 2    60   Output ~ 0
 SPI2_SCK
-Text GLabel 2900 4550 0    60   Output ~ 0
+Text GLabel 8500 2750 2    60   Output ~ 0
 SPI2_CS_B
-Text GLabel 8500 4050 2    60   Output ~ 0
+Text GLabel 8500 3350 2    60   Output ~ 0
 ~DISABLE_ESP
-Text GLabel 8500 2350 2    60   Output ~ 0
-ESP_BOOT_MODE
-Text GLabel 8500 2550 2    60   Input ~ 0
-ESP_DO
-Text GLabel 8500 2450 2    60   Output ~ 0
-ESP_DI
-$Comp
-L power:+BACKUP #PWR061
+$Comp
+L maxwell-rescue:+BACKUP-power #PWR061
 U 1 1 5A89D925
 P 2700 2650
@@
 Wire Wire Line
 	8500 4450 9250 4450
-NoConn ~ 8500 2650
-NoConn ~ 8500 2750
-NoConn ~ 8500 2850
 NoConn ~ 8500 3050
 NoConn ~ 8500 5150
@@
 NoConn ~ 2450 5400
 NoConn ~ 2650 5400
+Text GLabel 8500 2350 2    60   Output ~ 0
+BATT_SOURCE_DISABLE
 $EndSCHEMATC

Commit message: Updating hardware design.
Parts:
- C1, C2: symbol device:CP -> maxwell-rescue:CP-device
- J15: symbol conn:Conn_01x03 -> maxwell-rescue:Conn_01x03-conn
- U1: symbol coddingtonbear:MCP1501 -> maxwell-rescue:MCP1501-coddingtonbear
- Y1: symbol device:Crystal_GND23_Small -> maxwell-rescue:Crystal_GND23_Small-device
Changed lines of the file:
@@
 CAN_RX
 $Comp
-L coddingtonbear:MCP1501 U1
+L maxwell-rescue:MCP1501-coddingtonbear U1
 U 1 1 5A83FFBF
 P 7000 1500
@@
 	7800 1350 7550 1350
 $Comp
-L device:CP C2
+L maxwell-rescue:CP-device C2
 U 1 1 5A8463F3
 P 7900 1500
@@
 	6500 1300 6400 1300
 $Comp
-L device:CP C1
+L maxwell-rescue:CP-device C1
 U 1 1 5A848A15
 P 6250 1500
@@
 Connection ~ 6250 1650
 $Comp
-L device:Crystal_GND23_Small Y1
+L maxwell-rescue:Crystal_GND23_Small-device Y1
 U 1 1 5A8C64C3
 P 2550 5400
@@
 	2850 5150 2000 5150
 $Comp
-L conn:Conn_01x03 J15
+L maxwell-rescue:Conn_01x03-conn J15
 U 1 1 5A8B48F3
 P 9450 4350

Commit message: Preparing maxwell hardware for next revision.
Connections:
- net SPI2_CS_A: now also U7.16 (ADC1_IN2/ADC2_IN2/ADC3_IN2/TIM2_CH3/TIM5_CH3/USART2_TX/PA2); no longer U7.20 (ADC1_IN4/ADC2_IN4/DAC_OUT1/SPI1_NSS/USART2_CK/PA4)
- net SPI2_CS_B: now also U7.17 (ADC1_IN3/ADC2_IN3/ADC3_IN3/TIM2_CH4/TIM5_CH4/USART2_RX/PA3); no longer U7.21 (ADC1_IN5/ADC2_IN5/DAC_OUT2/SPI1_SCK/PA5)
- net DYNAMO_VOLTAGE: now reaches U7.24 (PC4/ADC1_IN14/ADC2_IN14)
- net DYNAMO_BUCK_VOLTAGE: now reaches U7.25 (PC5/ADC1_IN15/ADC2_IN15)
- net BATT_SOURCE_DISABLE renamed DYNAMO_SOURCE_DISABLE
- no-connect marks 8 -> 6
Changed lines of the file:
@@
 EESchema Schematic File Version 4
 LIBS:maxwell-cache
-EELAYER 26 0
+EELAYER 28 0
 EELAYER END
 $Descr A4 11693 8268
@@
 Wire Wire Line
 	2550 5550 2450 5550
-Text GLabel 8500 2650 2    60   Output ~ 0
+Text GLabel 8500 2450 2    60   Output ~ 0
 SPI2_CS_A
 Text GLabel 8500 5450 2    60   Output ~ 0
@@
 Text GLabel 8500 5250 2    60   Output ~ 0
 SPI2_SCK
-Text GLabel 8500 2750 2    60   Output ~ 0
+Text GLabel 8500 2550 2    60   Output ~ 0
 SPI2_CS_B
 Text GLabel 8500 3350 2    60   Output ~ 0
@@
 NoConn ~ 8500 3050
 NoConn ~ 8500 5150
-NoConn ~ 2900 4350
-NoConn ~ 2900 4450
 NoConn ~ 2900 4750
 NoConn ~ 2900 4850
@@
 NoConn ~ 2650 5400
 Text GLabel 8500 2350 2    60   Output ~ 0
-BATT_SOURCE_DISABLE
+DYNAMO_SOURCE_DISABLE
+Text GLabel 2900 4350 0    60   Input ~ 0
+DYNAMO_VOLTAGE
+Text GLabel 2900 4450 0    60   Input ~ 0
+DYNAMO_BUCK_VOLTAGE
 $EndSCHEMATC

Commit message: Updating hardware to reference the proper libraries; adding new parts to board to support switching from dynamo input to battery.
Parts:
- C10, C11, C12, C13, C6, C7, C8, C9, R10, R11, R33: footprint coddingtonbear/coddingtonbear.pretty:0805_Milling -> coddingtonbear:0805_Milling
- J15: footprint KiCad/Pin_Headers.pretty:Pin_Header_Straight_1x03_Pitch2.54mm -> coddingtonbear:JST_XH_B03B-XH-A_03x2.50mm_Straight_LargePads
- U1: footprint adamgreig/agg-kicad/agg.pretty:SOT-23-6 -> Package_TO_SOT_SMD:TSOT-23-6_HandSoldering
- Y1: footprint KiCad/Crystals.pretty:Crystal_SMD_SeikoEpson_MC306-4pin_8.0x3.2mm -> Crystal:Crystal_SMD_SeikoEpson_MC306-4Pin_8.0x3.2mm_HandSoldering
- Y2: footprint cpavlina/kicad-pcblib/smd-non-ipc.pretty:Abracon-ABM2 -> coddingtonbear:Abracon-ABM2
Changed lines of the file:
@@
 F 0 "Y2" V 2404 3731 50  0000 L CNN
 F 1 "8M" V 2495 3731 50  0000 L CNN
-F 2 "cpavlina/kicad-pcblib/smd-non-ipc.pretty:Abracon-ABM2" H 2450 3600 50  0001 C CNN
+F 2 "coddingtonbear:Abracon-ABM2" H 2450 3600 50  0001 C CNN
 F 3 "" H 2450 3600 50  0001 C CNN
 	1    2450 3600
@@
 F 0 "C6" V 2048 3450 50  0000 C CNN
 F 1 "22p" V 2139 3450 50  0000 C CNN
-F 2 "coddingtonbear/coddingtonbear.pretty:0805_Milling" H 2338 3300 50  0001 C CNN
+F 2 "coddingtonbear:0805_Milling" H 2338 3300 50  0001 C CNN
 F 3 "" H 2300 3450 50  0001 C CNN
 	1    2300 3450
@@
 F 0 "C7" V 2048 3750 50  0000 C CNN
 F 1 "22p" V 2139 3750 50  0000 C CNN
-F 2 "coddingtonbear/coddingtonbear.pretty:0805_Milling" H 2338 3600 50  0001 C CNN
+F 2 "coddingtonbear:0805_Milling" H 2338 3600 50  0001 C CNN
 F 3 "" H 2300 3750 50  0001 C CNN
 	1    2300 3750
@@
 F 0 "C8" V 2048 5250 50  0000 C CNN
 F 1 "22p" V 2139 5250 50  0000 C CNN
-F 2 "coddingtonbear/coddingtonbear.pretty:0805_Milling" H 2338 5100 50  0001 C CNN
+F 2 "coddingtonbear:0805_Milling" H 2338 5100 50  0001 C CNN
 F 3 "" H 2300 5250 50  0001 C CNN
 	1    2300 5250
@@
 F 0 "C9" V 2048 5550 50  0000 C CNN
 F 1 "22p" V 2139 5550 50  0000 C CNN
-F 2 "coddingtonbear/coddingtonbear.pretty:0805_Milling" H 2338 5400 50  0001 C CNN
+F 2 "coddingtonbear:0805_Milling" H 2338 5400 50  0001 C CNN
 F 3 "" H 2300 5550 50  0001 C CNN
 	1    2300 5550
@@
 F 0 "R10" V 2443 2250 50  0000 C CNN
 F 1 "10k" V 2534 2250 50  0000 C CNN
-F 2 "coddingtonbear/coddingtonbear.pretty:0805_Milling" V 2580 2250 50  0001 C CNN
+F 2 "coddingtonbear:0805_Milling" V 2580 2250 50  0001 C CNN
 F 3 "" H 2650 2250 50  0001 C CNN
 	1    2650 2250
@@
 F 0 "C10" H 5385 1454 50  0000 R CNN
 F 1 "100n" H 5385 1545 50  0000 R CNN
-F 2 "coddingtonbear/coddingtonbear.pretty:0805_Milling" H 5538 1350 50  0001 C CNN
+F 2 "coddingtonbear:0805_Milling" H 5538 1350 50  0001 C CNN
 F 3 "" H 5500 1500 50  0001 C CNN
 	1    5500 1500
@@
 F 0 "C11" H 5485 1454 50  0000 R CNN
 F 1 "100n" H 5485 1545 50  0000 R CNN
-F 2 "coddingtonbear/coddingtonbear.pretty:0805_Milling" H 5638 1350 50  0001 C CNN
+F 2 "coddingtonbear:0805_Milling" H 5638 1350 50  0001 C CNN
 F 3 "" H 5600 1500 50  0001 C CNN
 	1    5600 1500
@@
 F 0 "C12" H 5585 1454 50  0000 R CNN
 F 1 "100n" H 5585 1545 50  0000 R CNN
-F 2 "coddingtonbear/coddingtonbear.pretty:0805_Milling" H 5738 1350 50  0001 C CNN
+F 2 "coddingtonbear:0805_Milling" H 5738 1350 50  0001 C CNN
 F 3 "" H 5700 1500 50  0001 C CNN
 	1    5700 1500
@@
 F 0 "C13" H 5685 1454 50  0000 R CNN
 F 1 "100n" H 5685 1545 50  0000 R CNN
-F 2 "coddingtonbear/coddingtonbear.pretty:0805_Milling" H 5838 1350 50  0001 C CNN
+F 2 "coddingtonbear:0805_Milling" H 5838 1350 50  0001 C CNN
 F 3 "" H 5800 1500 50  0001 C CNN
 	1    5800 1500
@@
 F 0 "R33" V 2493 3600 50  0000 C CNN
 F 1 "1M" V 2584 3600 50  0000 C CNN
-F 2 "coddingtonbear/coddingtonbear.pretty:0805_Milling" V 2630 3600 50  0001 C CNN
+F 2 "coddingtonbear:0805_Milling" V 2630 3600 50  0001 C CNN
 F 3 "" H 2700 3600 50  0001 C CNN
 	1    2700 3600
@@
 F 0 "U1" H 7050 1013 60  0000 C CNN
 F 1 "MCP1501" H 7050 1119 60  0000 C CNN
-F 2 "adamgreig/agg-kicad/agg.pretty:SOT-23-6" H 7000 1500 60  0001 C CNN
+F 2 "Package_TO_SOT_SMD:TSOT-23-6_HandSoldering" H 7000 1500 60  0001 C CNN
 F 3 "" H 7000 1500 60  0001 C CNN
 	1    7000 1500
@@
 F 0 "R11" V 5843 1250 50  0000 C CNN
 F 1 "50" V 5934 1250 50  0000 C CNN
-F 2 "coddingtonbear/coddingtonbear.pretty:0805_Milling" V 5980 1250 50  0001 C CNN
+F 2 "coddingtonbear:0805_Milling" V 5980 1250 50  0001 C CNN
 F 3 "" H 6050 1250 50  0001 C CNN
 	1    6050 1250
@@
 F 0 "Y1" V 2504 5566 50  0000 L CNN
 F 1 "32.768k" V 2595 5566 50  0000 L CNN
-F 2 "KiCad/Crystals.pretty:Crystal_SMD_SeikoEpson_MC306-4pin_8.0x3.2mm" H 2550 5400 50  0001 C CNN
+F 2 "Crystal:Crystal_SMD_SeikoEpson_MC306-4Pin_8.0x3.2mm_HandSoldering" H 2550 5400 50  0001 C CNN
 F 3 "" H 2550 5400 50  0001 C CNN
 	1    2550 5400
@@
 F 0 "J15" H 9529 4392 50  0000 L CNN
 F 1 "GPIO" H 9529 4301 50  0000 L CNN
-F 2 "KiCad/Pin_Headers.pretty:Pin_Header_Straight_1x03_Pitch2.54mm" H 9450 4350 50  0001 C CNN
+F 2 "coddingtonbear:JST_XH_B03B-XH-A_03x2.50mm_Straight_LargePads" H 9450 4350 50  0001 C CNN
 F 3 "~" H 9450 4350 50  0001 C CNN
 	1    9450 4350
