File: hardware/maxwell/microcontroller.sch (KiCad schematic (older format))
At the start: 18 parts, among them J15 GPIO, U1 MCP1501, U7 STM32F103RETx, Y1 32.768k, Y2 8M

Commit message: v1.5 ready for production.
Parts:
- removed C1, C2: 2.2u, coddingtonbear:CP_Tantalum_Case-C_EIA-6032-28_Milling, symbol maxwell-rescue:CP-device
- removed J15: GPIO, coddingtonbear:JST_XH_B03B-XH-A_03x2.50mm_Straight_LargePads, symbol maxwell-rescue:Conn_01x03-conn
- removed R11: 50, coddingtonbear:0805_Milling, symbol maxwell-rescue:R-RESCUE-maxwell
- removed U1: MCP1501, Package_TO_SOT_SMD:TSOT-23-6_HandSoldering, symbol maxwell-rescue:MCP1501-coddingtonbear
- U7: footprint kicad-castellated-breakouts:QFP64-1.27MM-CASTELLATED-VERS -> kicad-castellated-breakouts:QFP64-1.27MM-CASTELLATED
Connections:
- net BATT_VOLTAGE is gone; now on net SPEED: U7.8 (PC0/ADC1_IN10/ADC2_IN10/ADC3_IN10)
- net DYNAMO_SOURCE_DISABLE is gone; now on net SPI2_CS_B: U7.15 (ADC1_IN1/ADC2_IN1/ADC3_IN1/TIM2_CH2/TIM5_CH2/USART2_RTS/PA1)
- net DYNAMO_VOLTAGE is gone; now on net ENABLE_BATT_POWER: U7.24 (PC4/ADC1_IN14/ADC2_IN14)
- net +3V3: now also U7.13 (VDDA)
- net BUZZER: now also U7.17 (ADC1_IN3/ADC2_IN3/ADC3_IN3/TIM2_CH4/TIM5_CH4/USART2_RX/PA3); no longer U7.45 (CAN_TX/TIM1_ETR/USART1_RTS/USB_DP/PA12)
- net CAN_DISABLE: now also U7.56 (SPI1_MISO/SPI3_MISO/SYS_NJTRST/TIM3_CH1/PB4); no longer U7.11 (PC3/ADC1_IN13/ADC2_IN13/ADC3_IN13)
- net ENABLE_BATT_POWER: no longer U7.26 (ADC1_IN8/ADC2_IN8/TIM1_CH2N/TIM3_CH3/TIM8_CH2N/PB0)
- net POWER_ON: now also U7.55 (I2S3_CK/SPI1_SCK/SPI3_SCK/SYS_JTDO-TRACESWO/TIM2_CH2/PB3); no longer U7.50 (ADC1_EXTI15/ADC2_EXTI15/I2S3_WS/SPI1_NSS/SPI3_NSS/SYS_JTDI/TIM2_CH1/TIM2_ETR/PA15)
- net SPEED: no longer U7.14 (ADC1_IN0/ADC2_IN0/ADC3_IN0/SYS_WKUP/TIM2_CH1/TIM2_ETR/TIM5_CH1/TIM8_ETR/USART2_CTS/PA0)
- net SPI2_CS_B: no longer U7.17 (ADC1_IN3/ADC2_IN3/ADC3_IN3/TIM2_CH4/TIM5_CH4/USART2_RX/PA3)
- net ~DISABLE_ESP: now also U7.38 (PC7/I2S3_MCK/SDIO_D7/TIM3_CH2/TIM8_CH2); no longer U7.44 (ADC1_EXTI11/ADC2_EXTI11/CAN_RX/TIM1_CH4/USART1_CTS/USB_DM/PA11)
- net CURRENT_SENSE: no longer names the net of U7.9 (PC1/ADC1_IN11/ADC2_IN11/ADC3_IN11)
- net DYNAMO_BUCK_VOLTAGE: no longer names the net of U7.25 (PC5/ADC1_IN15/ADC2_IN15)
- net GPS_DI: no longer names the net of U7.29 (I2C2_SCL/TIM2_CH3/USART3_TX/PB10)
- net GPS_DO: no longer names the net of U7.30 (ADC1_EXTI11/ADC2_EXTI11/I2C2_SDA/TIM2_CH4/USART3_RX/PB11)
- net ~BATT_CHARGE_ENABLE: no longer names the net of U7.2 (PC13/RTC_OUT/RTC_TAMPER)
- net ~BATT_CHARGING: no longer names the net of U7.10 (PC2/ADC1_IN12/ADC2_IN12/ADC3_IN12)
- new net SPI2_CS_C: U7.14 (ADC1_IN0/ADC2_IN0/ADC3_IN0/SYS_WKUP/TIM2_CH1/TIM2_ETR/TIM5_CH1/TIM8_ETR/USART2_CTS/PA0)
- no-connect marks 6 -> 9
Changed lines of the file:
@@
 EESchema Schematic File Version 4
 LIBS:maxwell-cache
-EELAYER 28 0
+EELAYER 29 0
 EELAYER END
 $Descr A4 11693 8268
@@
 F 0 "U7" H 5700 6028 50  0000 C CNN
 F 1 "STM32F103RETx" H 5700 5937 50  0000 C CNN
-F 2 "kicad-castellated-breakouts:QFP64-1.27MM-CASTELLATED-VERS" H 8400 5725 50  0001 R TNN
+F 2 "kicad-castellated-breakouts:QFP64-1.27MM-CASTELLATED" H 8400 5725 50  0001 R TNN
 F 3 "" H 5700 3850 50  0001 C CNN
 	1    5700 3850
@@
 Wire Wire Line
 	5500 1350 5600 1350
-Connection ~ 5800 1350
 Connection ~ 5700 1350
 Connection ~ 5600 1350
@@
 Text GLabel 8500 3650 2    60   BiDi ~ 0
 SWCLK
-Text GLabel 8500 2250 2    60   Input ~ 0
+Text GLabel 2900 3950 0    60   Input ~ 0
 SPEED
-Text GLabel 2900 4150 0    60   Input ~ 0
-~BATT_CHARGING
-Text GLabel 8500 3750 2    60   Input ~ 0
+Text GLabel 8500 4250 2    60   Input ~ 0
 POWER_ON
 Text GLabel 8500 3150 2    60   Output ~ 0
@@
 Text GLabel 2900 4550 0    60   Output ~ 0
 BT_KEY
-Text GLabel 2900 4050 0    60   Input ~ 0
-CURRENT_SENSE
-Text GLabel 2900 3950 0    60   Input ~ 0
-BATT_VOLTAGE
-Text GLabel 8500 3450 2    60   Output ~ 0
+Text GLabel 8500 2550 2    60   Output ~ 0
 BUZZER
 Text GLabel 8500 2950 2    60   Output ~ 0
@@
 	2850 1850 2850 2250
 Connection ~ 2850 2250
-Text GLabel 8500 3950 2    60   Output ~ 0
+Text GLabel 2900 4350 0    60   Output ~ 0
 ENABLE_BATT_POWER
 $Comp
@@
 	2800 3650 2900 3650
 Connection ~ 2700 3750
-Text GLabel 2900 4250 0    60   Output ~ 0
+Text GLabel 8500 4350 2    60   Output ~ 0
 CAN_DISABLE
-Text GLabel 2000 5150 0    60   Output ~ 0
-~BATT_CHARGE_ENABLE
 Wire Wire Line
 	2150 3600 2150 3750
@@
 Text GLabel 8500 4750 2    60   Input ~ 0
 CAN_RX
-$Comp
-L maxwell-rescue:MCP1501-coddingtonbear U1
-U 1 1 5A83FFBF
-P 7000 1500
-F 0 "U1" H 7050 1013 60  0000 C CNN
-F 1 "MCP1501" H 7050 1119 60  0000 C CNN
-F 2 "Package_TO_SOT_SMD:TSOT-23-6_HandSoldering" H 7000 1500 60  0001 C CNN
-F 3 "" H 7000 1500 60  0001 C CNN
-	1    7000 1500
-	-1   0    0    1
-$EndComp
-Wire Wire Line
-	6550 1650 6250 1650
-$Comp
-L maxwell-rescue:+3V3-RESCUE-maxwell #PWR022
-U 1 1 5A841B1D
-P 8200 1650
-F 0 "#PWR022" H 8200 1500 50  0001 C CNN
-F 1 "+3V3" H 8215 1823 50  0000 C CNN
-F 2 "" H 8200 1650 50  0001 C CNN
-F 3 "" H 8200 1650 50  0001 C CNN
-	1    8200 1650
-	1    0    0    -1
-$EndComp
-Wire Wire Line
-	7400 1300 7550 1300
-Wire Wire Line
-	7550 1300 7550 1350
-Wire Wire Line
-	7550 1400 7400 1400
-Wire Wire Line
-	7400 1500 7550 1500
-Wire Wire Line
-	7550 1500 7550 1400
-Connection ~ 7550 1400
-Connection ~ 7550 1350
-Wire Wire Line
-	7550 1350 7550 1400
-$Comp
-L maxwell-rescue:GND-RESCUE-maxwell #PWR030
-U 1 1 5A845E73
-P 7800 1350
-F 0 "#PWR030" H 7800 1100 50  0001 C CNN
-F 1 "GND" H 7805 1177 50  0000 C CNN
-F 2 "" H 7800 1350 50  0001 C CNN
-F 3 "" H 7800 1350 50  0001 C CNN
-	1    7800 1350
-	-1   0    0    1
-$EndComp
-Wire Wire Line
-	7800 1350 7550 1350
-$Comp
-L maxwell-rescue:CP-device C2
-U 1 1 5A8463F3
-P 7900 1500
-F 0 "C2" H 7782 1454 50  0000 R CNN
-F 1 "2.2u" H 7782 1545 50  0000 R CNN
-F 2 "coddingtonbear:CP_Tantalum_Case-C_EIA-6032-28_Milling" H 7938 1350 50  0001 C CNN
-F 3 "" H 7900 1500 50  0001 C CNN
-	1    7900 1500
-	-1   0    0    1
-$EndComp
-Connection ~ 7900 1650
-Wire Wire Line
-	7900 1650 8200 1650
-Wire Wire Line
-	7900 1350 7800 1350
-Wire Wire Line
-	7400 1650 7900 1650
-Connection ~ 7800 1350
-$Comp
-L maxwell-rescue:+3V3-RESCUE-maxwell #PWR031
-U 1 1 5A847782
-P 6400 1300
-F 0 "#PWR031" H 6400 1150 50  0001 C CNN
-F 1 "+3V3" H 6415 1473 50  0000 C CNN
-F 2 "" H 6400 1300 50  0001 C CNN
-F 3 "" H 6400 1300 50  0001 C CNN
-	1    6400 1300
-	1    0    0    -1
-$EndComp
-Wire Wire Line
-	6500 1300 6400 1300
-$Comp
-L maxwell-rescue:CP-device C1
-U 1 1 5A848A15
-P 6250 1500
-F 0 "C1" H 6132 1454 50  0000 R CNN
-F 1 "2.2u" H 6132 1545 50  0000 R CNN
-F 2 "coddingtonbear:CP_Tantalum_Case-C_EIA-6032-28_Milling" H 6288 1350 50  0001 C CNN
-F 3 "" H 6250 1500 50  0001 C CNN
-	1    6250 1500
-	-1   0    0    1
-$EndComp
-$Comp
-L maxwell-rescue:R-RESCUE-maxwell R11
-U 1 1 5A848A7F
-P 6050 1250
-F 0 "R11" V 5843 1250 50  0000 C CNN
-F 1 "50" V 5934 1250 50  0000 C CNN
-F 2 "coddingtonbear:0805_Milling" V 5980 1250 50  0001 C CNN
-F 3 "" H 6050 1250 50  0001 C CNN
-	1    6050 1250
-	0    1    1    0
-$EndComp
-Wire Wire Line
-	6250 1350 6250 1250
-Wire Wire Line
-	6250 1250 6200 1250
-Wire Wire Line
-	5900 1250 5800 1250
-Wire Wire Line
-	5800 1250 5800 1350
-Wire Wire Line
-	5900 1850 6250 1850
-Wire Wire Line
-	6250 1850 6250 1650
-Connection ~ 6250 1650
 $Comp
 L maxwell-rescue:Crystal_GND23_Small-device Y1
@@
 Text GLabel 8500 5250 2    60   Output ~ 0
 SPI2_SCK
-Text GLabel 8500 2550 2    60   Output ~ 0
+Text GLabel 8500 2350 2    60   Output ~ 0
 SPI2_CS_B
-Text GLabel 8500 3350 2    60   Output ~ 0
+Text GLabel 2900 4650 0    60   Output ~ 0
 ~DISABLE_ESP
 $Comp
@@
 Wire Wire Line
 	2900 2650 2700 2650
-Text GLabel 8500 5050 2    60   Input ~ 0
-GPS_DO
-Text GLabel 8500 4950 2    60   Output ~ 0
-GPS_DI
 Wire Wire Line
 	2800 3850 2850 3850
@@
 Wire Wire Line
 	2900 5250 2850 5250
-Wire Wire Line
-	2850 5250 2850 5150
-Wire Wire Line
-	2850 5150 2000 5150
-$Comp
-L maxwell-rescue:Conn_01x03-conn J15
-U 1 1 5A8B48F3
-P 9450 4350
-F 0 "J15" H 9529 4392 50  0000 L CNN
-F 1 "GPIO" H 9529 4301 50  0000 L CNN
-F 2 "coddingtonbear:JST_XH_B03B-XH-A_03x2.50mm_Straight_LargePads" H 9450 4350 50  0001 C CNN
-F 3 "~" H 9450 4350 50  0001 C CNN
-	1    9450 4350
-	1    0    0    -1
-$EndComp
-Wire Wire Line
-	8500 4250 9250 4250
-Wire Wire Line
-	9250 4350 8500 4350
-Wire Wire Line
-	8500 4450 9250 4450
 NoConn ~ 8500 3050
 NoConn ~ 8500 5150
@@
 NoConn ~ 2450 5400
 NoConn ~ 2650 5400
-Text GLabel 8500 2350 2    60   Output ~ 0
-DYNAMO_SOURCE_DISABLE
-Text GLabel 2900 4350 0    60   Input ~ 0
-DYNAMO_VOLTAGE
-Text GLabel 2900 4450 0    60   Input ~ 0
-DYNAMO_BUCK_VOLTAGE
+NoConn ~ 8500 2850
+NoConn ~ 8500 2750
+NoConn ~ 8500 2650
+Wire Wire Line
+	5800 1750 5900 1750
+Wire Wire Line
+	5900 1750 5900 1850
+Text GLabel 8500 2250 2    60   Output ~ 0
+SPI2_CS_C
 $EndSCHEMATC
