File: hardware/maxwell/rectification.sch (KiCad schematic (older format))
At the start: 23 parts, among them J19 Interconnect (Rect), Q6 DMG2302UK, Q7 DMG2302UK, Q8 DMG2302UK, Q9 DMG2302UK, U15 LM74670-Q1, U16 LM74670-Q1, U17 LM74670-Q1, U18 LM74670-Q1, U19 LT3086IR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

Commit message: Missing connection from diode controller to VDYN+; bodged.
Connections:
- net at C29.1, Q8.3 (D), Q9.3 (D)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: now also U18.8 (Cathode)
Changed lines of the file:
@@
 	6100 2950 7050 2950
 Connection ~ 6100 2950
-Wire Wire Line
-	6100 2950 6100 3050
 Connection ~ 7050 2950
 Wire Wire Line
@@
 	1    0    0    -1
 $EndComp
+Wire Wire Line
+	6100 2950 6100 3150
 $EndSCHEMATC

Commit message: Maxwell v1.9.2
Over the last month, I've melted the voltage cap zeners
off of the rectifier board. This is not great; they serve
an essential purpose in preventing the mosfets and active
rectifiers behind it from being exposed to an overvoltage
situation and burning out (which has happened to at least
one mosfet).

* Uses much bigger DO-201AE package through-hole diodes.
  These should be able to dissapate a lot more heat, and
  if they do heat up the solder enough to begin melting
  at least they won't be able to fall out of position.
* Adds a P-Ch mosfet between the rectifier and capacitor;
  this should allow me to programmatically turn off the
  dynamo power source when I'm travelling very slowly
  or heading uphill.
Parts:
- added Q11: Q_PMOS_GDSD, Package_TO_SOT_SMD:SOT-223, symbol Device:Q_PMOS_GDSD
- added R41: 10k, coddingtonbear:0805_Milling, symbol maxwell-rescue:R-RESCUE-maxwell
- D3, D4: footprint coddingtonbear:D_SOD-123_LargePads -> Diode_THT:D_DO-201AE_P15.24mm_Horizontal
Connections:
- net labels added: DISABLE_DYNAMO
- net labels removed: VDYN_C
- wire segments 79 -> 88
Other:
- moved on the sheet: C29, R15, R17
Changed lines of the file:
@@
 F 0 "D3" V 2604 2379 50  0000 L CNN
 F 1 "18V" V 2695 2379 50  0000 L CNN
-F 2 "coddingtonbear:D_SOD-123_LargePads" H 2650 2300 50  0001 C CNN
+F 2 "Diode_THT:D_DO-201AE_P15.24mm_Horizontal" H 2650 2300 50  0001 C CNN
 F 3 "~" H 2650 2300 50  0001 C CNN
 	1    2650 2300
@@
 F 0 "D4" V 2696 2521 50  0000 R CNN
 F 1 "18V" V 2605 2521 50  0000 R CNN
-F 2 "coddingtonbear:D_SOD-123_LargePads" H 2650 2600 50  0001 C CNN
+F 2 "Diode_THT:D_DO-201AE_P15.24mm_Horizontal" H 2650 2600 50  0001 C CNN
 F 3 "~" H 2650 2600 50  0001 C CNN
 	1    2650 2600
 	0    -1   -1   0
 $EndComp
-Text GLabel 8050 3650 3    60   Output ~ 0
+Text GLabel 8400 3650 3    60   Output ~ 0
 DYNAMO_VOLTAGE_C
 $Comp
 L maxwell-rescue:R-RESCUE-maxwell R?
 U 1 1 5C7ACBC0
-P 7800 3300
+P 8150 3300
 AR Path="/5A1FEBCF/5C7ACBC0" Ref="R?"  Part="1"
 AR Path="/5A1FEBCF/5C7831A2/5C7ACBC0" Ref="R15"  Part="1"
-F 0 "R15" H 7870 3346 50  0000 L CNN
-F 1 "20k" H 7870 3255 50  0000 L CNN
-F 2 "coddingtonbear:0805_Milling" V 7730 3300 50  0001 C CNN
-F 3 "" H 7800 3300 50  0001 C CNN
-	1    7800 3300
+F 0 "R15" H 8220 3346 50  0000 L CNN
+F 1 "20k" H 8220 3255 50  0000 L CNN
+F 2 "coddingtonbear:0805_Milling" V 8080 3300 50  0001 C CNN
+F 3 "" H 8150 3300 50  0001 C CNN
+	1    8150 3300
 	1    0    0    -1
 $EndComp
@@
 L maxwell-rescue:R-RESCUE-maxwell R?
 U 1 1 5C7ACBC7
-P 7800 3750
+P 8150 3750
 AR Path="/5A1FEBCF/5C7ACBC7" Ref="R?"  Part="1"
 AR Path="/5A1FEBCF/5C7831A2/5C7ACBC7" Ref="R17"  Part="1"
-F 0 "R17" H 7870 3796 50  0000 L CNN
-F 1 "1470" H 7870 3705 50  0000 L CNN
-F 2 "coddingtonbear:0805_Milling" V 7730 3750 50  0001 C CNN
-F 3 "" H 7800 3750 50  0001 C CNN
-	1    7800 3750
+F 0 "R17" H 8220 3796 50  0000 L CNN
+F 1 "1470" H 8220 3705 50  0000 L CNN
+F 2 "coddingtonbear:0805_Milling" V 8080 3750 50  0001 C CNN
+F 3 "" H 8150 3750 50  0001 C CNN
+	1    8150 3750
 	-1   0    0    1
 $EndComp
@@
 	3800 2950 3500 2950
 Wire Wire Line
-	7050 2950 7250 2950
-Wire Wire Line
-	7800 3150 7800 2950
-Connection ~ 7250 2950
-Wire Wire Line
 	4750 1650 6100 1650
 Wire Wire Line
@@
 L Device:CP_Small C29
 U 1 1 5C7CB665
-P 7250 3050
-F 0 "C29" H 7338 3096 50  0000 L CNN
-F 1 "6000uF" H 7338 3005 50  0000 L CNN
-F 2 "coddingtonbear:JST_XH_B02B-XH-A_02x2.50mm_Straight_LargePads" H 7250 3050 50  0001 C CNN
-F 3 "~" H 7250 3050 50  0001 C CNN
-	1    7250 3050
-	1    0    0    -1
-$EndComp
-Wire Wire Line
-	7800 3450 7800 3500
-Wire Wire Line
-	7800 2950 7250 2950
-Wire Wire Line
-	7800 3500 8050 3500
-Wire Wire Line
-	8050 3500 8050 3650
-Connection ~ 7800 3500
-Wire Wire Line
-	7800 3500 7800 3600
+P 7700 3050
+F 0 "C29" H 7788 3096 50  0000 L CNN
+F 1 "6000uF" H 7788 3005 50  0000 L CNN
+F 2 "coddingtonbear:JST_XH_B02B-XH-A_02x2.50mm_Straight_LargePads" H 7700 3050 50  0001 C CNN
+F 3 "~" H 7700 3050 50  0001 C CNN
+	1    7700 3050
+	1    0    0    -1
+$EndComp
+Wire Wire Line
+	8150 3450 8150 3500
+Wire Wire Line
+	8150 3500 8400 3500
+Wire Wire Line
+	8400 3500 8400 3650
+Connection ~ 8150 3500
+Wire Wire Line
+	8150 3500 8150 3600
 $Comp
 L coddingtonbear:LT3086IR U19
@@
 Wire Wire Line
 	8550 2950 8300 2950
-Connection ~ 7800 2950
 Wire Wire Line
 	8550 3100 8300 3100
@@
 	8300 3100 8300 2950
 Connection ~ 8300 2950
-Wire Wire Line
-	8300 2950 7800 2950
 Wire Wire Line
 	8550 3300 8550 3550
@@
 L coddingtonbear:GND_C #PWR0166
 U 1 1 5CA9C407
-P 7800 3900
-F 0 "#PWR0166" H 7800 3650 50  0001 C CNN
-F 1 "GND_C" H 7805 3727 50  0000 C CNN
-F 2 "" H 7800 3900 50  0001 C CNN
-F 3 "" H 7800 3900 50  0001 C CNN
-	1    7800 3900
+P 8150 3900
+F 0 "#PWR0166" H 8150 3650 50  0001 C CNN
+F 1 "GND_C" H 8155 3727 50  0000 C CNN
+F 2 "" H 8150 3900 50  0001 C CNN
+F 3 "" H 8150 3900 50  0001 C CNN
+	1    8150 3900
 	1    0    0    -1
 $EndComp
@@
 Wire Wire Line
 	8950 3550 9150 3550
-Text GLabel 9850 2800 1    60   Output ~ 0
-VDYN_C
-Wire Wire Line
-	9850 2950 9850 2800
-Connection ~ 9850 2950
-Text GLabel 1600 2750 3    60   Input ~ 0
-VDYN_C
 Text GLabel 1500 2750 3    60   Input ~ 0
 DYNAMO_VOLTAGE_C
@@
 L coddingtonbear:GND_C #PWR0178
 U 1 1 5CC23766
-P 7250 3150
-F 0 "#PWR0178" H 7250 2900 50  0001 C CNN
-F 1 "GND_C" H 7255 2977 50  0000 C CNN
-F 2 "" H 7250 3150 50  0001 C CNN
-F 3 "" H 7250 3150 50  0001 C CNN
-	1    7250 3150
+P 7700 3150
+F 0 "#PWR0178" H 7700 2900 50  0001 C CNN
+F 1 "GND_C" H 7705 2977 50  0000 C CNN
+F 2 "" H 7700 3150 50  0001 C CNN
+F 3 "" H 7700 3150 50  0001 C CNN
+	1    7700 3150
 	1    0    0    -1
 $EndComp
 Wire Wire Line
 	6100 2950 6100 3150
+Wire Wire Line
+	7700 2950 8150 2950
+Wire Wire Line
+	8150 3150 8150 2950
+Connection ~ 8150 2950
+Wire Wire Line
+	8150 2950 8300 2950
+$Comp
+L Device:Q_PMOS_GDSD Q11
+U 1 1 5CA84A4C
+P 7250 2850
+F 0 "Q11" V 7582 2850 50  0000 C CNN
+F 1 "Q_PMOS_GDSD" V 7673 2850 50  0000 C CNN
+F 2 "Package_TO_SOT_SMD:SOT-223" H 7450 2950 50  0001 C CNN
+F 3 "~" H 7250 2850 50  0001 C CNN
+	1    7250 2850
+	0    1    1    0
+$EndComp
+$Comp
+L maxwell-rescue:R-RESCUE-maxwell R?
+U 1 1 5CA8831A
+P 7600 2600
+AR Path="/5A1FEBCF/5CA8831A" Ref="R?"  Part="1"
+AR Path="/5A1FEBCF/5C7831A2/5CA8831A" Ref="R41"  Part="1"
+F 0 "R41" H 7670 2646 50  0000 L CNN
+F 1 "10k" H 7670 2555 50  0000 L CNN
+F 2 "coddingtonbear:0805_Milling" V 7530 2600 50  0001 C CNN
+F 3 "" H 7600 2600 50  0001 C CNN
+	1    7600 2600
+	0    1    1    0
+$EndComp
+$Comp
+L coddingtonbear:GND_C #PWR0194
+U 1 1 5CA8840C
+P 7900 2650
+F 0 "#PWR0194" H 7900 2400 50  0001 C CNN
+F 1 "GND_C" H 7905 2477 50  0000 C CNN
+F 2 "" H 7900 2650 50  0001 C CNN
+F 3 "" H 7900 2650 50  0001 C CNN
+	1    7900 2650
+	1    0    0    -1
+$EndComp
+Wire Wire Line
+	7250 2650 7250 2600
+Wire Wire Line
+	7250 2600 7450 2600
+Wire Wire Line
+	7750 2600 7900 2600
+Wire Wire Line
+	7900 2600 7900 2650
+Text GLabel 1600 2750 3    60   Output ~ 0
+DISABLE_DYNAMO
+Wire Wire Line
+	1200 2250 1200 2750
+Text GLabel 7350 2450 2    60   Input ~ 0
+DISABLE_DYNAMO
+Wire Wire Line
+	7350 2450 7250 2450
+Wire Wire Line
+	7250 2450 7250 2600
+Connection ~ 7250 2600
+Wire Wire Line
+	7450 3050 7500 3050
+Wire Wire Line
+	7500 3050 7500 2950
+Wire Wire Line
+	7500 2950 7700 2950
+Connection ~ 7700 2950
+Wire Wire Line
+	7450 2950 7500 2950
+Connection ~ 7500 2950
 $EndSCHEMATC

Commit message: Maxwell Remote v1.9.3
* Uses LT3086IR's SHDN pin instead of a separate mosfet.
* Minor board layout and size changes.
Parts:
- removed Q11: Q_PMOS_GDSD, Package_TO_SOT_SMD:SOT-223, symbol Device:Q_PMOS_GDSD
Connections:
- net labels added: DYNAMO_REG_OUT, ~DISABLE_DYNAMO
- net labels removed: DISABLE_DYNAMO
- wire segments 88 -> 84
Changed lines of the file:
@@
 	0    -1   -1   0
 $EndComp
-Text GLabel 8400 3650 3    60   Output ~ 0
+Text GLabel 7750 3600 3    60   Output ~ 0
 DYNAMO_VOLTAGE_C
 $Comp
@@
 AR Path="/5A1FEBCF/5C7ACBC0" Ref="R?"  Part="1"
 AR Path="/5A1FEBCF/5C7831A2/5C7ACBC0" Ref="R15"  Part="1"
-F 0 "R15" H 8220 3346 50  0000 L CNN
-F 1 "20k" H 8220 3255 50  0000 L CNN
+F 0 "R15" H 7950 3350 50  0000 L CNN
+F 1 "20k" H 7950 3250 50  0000 L CNN
 F 2 "coddingtonbear:0805_Milling" V 8080 3300 50  0001 C CNN
 F 3 "" H 8150 3300 50  0001 C CNN
@@
 	1    0    0    -1
 $EndComp
-Wire Wire Line
-	8150 3450 8150 3500
-Wire Wire Line
-	8150 3500 8400 3500
-Wire Wire Line
-	8400 3500 8400 3650
-Connection ~ 8150 3500
-Wire Wire Line
-	8150 3500 8150 3600
 $Comp
 L coddingtonbear:LT3086IR U19
@@
 	1    0    0    -1
 $EndComp
-Wire Wire Line
-	8550 2950 8300 2950
-Wire Wire Line
-	8550 3100 8300 3100
-Wire Wire Line
-	8300 3100 8300 2950
-Connection ~ 8300 2950
 Wire Wire Line
 	8550 3300 8550 3550
@@
 	8150 3150 8150 2950
 Connection ~ 8150 2950
-Wire Wire Line
-	8150 2950 8300 2950
-$Comp
-L Device:Q_PMOS_GDSD Q11
-U 1 1 5CA84A4C
-P 7250 2850
-F 0 "Q11" V 7582 2850 50  0000 C CNN
-F 1 "Q_PMOS_GDSD" V 7673 2850 50  0000 C CNN
-F 2 "Package_TO_SOT_SMD:SOT-223" H 7450 2950 50  0001 C CNN
-F 3 "~" H 7250 2850 50  0001 C CNN
-	1    7250 2850
-	0    1    1    0
-$EndComp
+Text GLabel 1200 2750 3    60   Output ~ 0
+~DISABLE_DYNAMO
+Wire Wire Line
+	1200 2250 1200 2750
+Text GLabel 8450 3900 3    60   Input ~ 0
+~DISABLE_DYNAMO
+Wire Wire Line
+	8150 3450 8150 3500
+Wire Wire Line
+	7750 3600 7750 3500
+Wire Wire Line
+	7750 3500 8150 3500
+Connection ~ 8150 3500
+Wire Wire Line
+	8150 3500 8150 3600
+Wire Wire Line
+	8150 2950 8250 2950
+Wire Wire Line
+	8450 3100 8550 3100
+Wire Wire Line
+	7700 2950 7050 2950
+Connection ~ 7700 2950
+Text GLabel 9900 2800 2    60   Output ~ 0
+DYNAMO_REG_OUT
+Text GLabel 1600 2750 3    60   Input ~ 0
+DYNAMO_REG_OUT
+Wire Wire Line
+	9900 2800 9850 2800
+Wire Wire Line
+	9850 2800 9850 2950
+Connection ~ 9850 2950
 $Comp
 L maxwell-rescue:R-RESCUE-maxwell R?
-U 1 1 5CA8831A
-P 7600 2600
-AR Path="/5A1FEBCF/5CA8831A" Ref="R?"  Part="1"
-AR Path="/5A1FEBCF/5C7831A2/5CA8831A" Ref="R41"  Part="1"
-F 0 "R41" H 7670 2646 50  0000 L CNN
-F 1 "10k" H 7670 2555 50  0000 L CNN
-F 2 "coddingtonbear:0805_Milling" V 7530 2600 50  0001 C CNN
-F 3 "" H 7600 2600 50  0001 C CNN
-	1    7600 2600
-	0    1    1    0
-$EndComp
-$Comp
-L coddingtonbear:GND_C #PWR0194
-U 1 1 5CA8840C
-P 7900 2650
-F 0 "#PWR0194" H 7900 2400 50  0001 C CNN
-F 1 "GND_C" H 7905 2477 50  0000 C CNN
-F 2 "" H 7900 2650 50  0001 C CNN
-F 3 "" H 7900 2650 50  0001 C CNN
-	1    7900 2650
-	1    0    0    -1
-$EndComp
-Wire Wire Line
-	7250 2650 7250 2600
-Wire Wire Line
-	7250 2600 7450 2600
-Wire Wire Line
-	7750 2600 7900 2600
-Wire Wire Line
-	7900 2600 7900 2650
-Text GLabel 1600 2750 3    60   Output ~ 0
-DISABLE_DYNAMO
-Wire Wire Line
-	1200 2250 1200 2750
-Text GLabel 7350 2450 2    60   Input ~ 0
-DISABLE_DYNAMO
-Wire Wire Line
-	7350 2450 7250 2450
-Wire Wire Line
-	7250 2450 7250 2600
-Connection ~ 7250 2600
-Wire Wire Line
-	7450 3050 7500 3050
-Wire Wire Line
-	7500 3050 7500 2950
-Wire Wire Line
-	7500 2950 7700 2950
-Connection ~ 7700 2950
-Wire Wire Line
-	7450 2950 7500 2950
-Connection ~ 7500 2950
+U 1 1 5CAC37BE
+P 8250 3650
+AR Path="/5A1FEBCF/5CAC37BE" Ref="R?"  Part="1"
+AR Path="/5A1FEBCF/5C7831A2/5CAC37BE" Ref="R41"  Part="1"
+F 0 "R41" H 8300 3700 50  0000 L CNN
+F 1 "10k" H 8300 3600 50  0000 L CNN
+F 2 "coddingtonbear:0805_Milling" V 8180 3650 50  0001 C CNN
+F 3 "" H 8250 3650 50  0001 C CNN
+	1    8250 3650
+	1    0    0    -1
+$EndComp
+Wire Wire Line
+	8250 3500 8250 2950
+Connection ~ 8250 2950
+Wire Wire Line
+	8250 2950 8550 2950
+Wire Wire Line
+	8450 3100 8450 3800
+Wire Wire Line
+	8250 3800 8450 3800
+Connection ~ 8450 3800
+Wire Wire Line
+	8450 3800 8450 3900
 $EndSCHEMATC

Commit message: Maxwell Remote v1.9.4
It occurred to me that were I to turn off the
regulator, the voltage would just have to be
burned off in the Zener diodes because the dynamo
will just ratchet the voltage up as high as it could.
Really -- I should just use a triac to turn off
the dynamo.

* Adds a (default-enabled) triac for switching
  the dynamo on and off.
Parts:
- added U22: BTA20-700CWRG, Package_TO_SOT_THT:TO-220-3_Vertical, symbol custom:TRIAC_AAG
- R41: value 10k -> 340
Changed lines of the file:
@@
 	3800 3700 3800 4300
-Wire Wire Line
-	3800 1650 2650 1650
-Wire Wire Line
-	2650 1650 2650 2150
-Connection ~ 3800 1650
 Wire Wire Line
 	2650 2750 2650 4300
@@
 Text GLabel 1100 2750 3    60   Output ~ 0
 V_AC-
-Text GLabel 2650 2150 0    60   Input ~ 0
+Text GLabel 1950 1650 0    60   Input ~ 0
 V_AC+
 Text GLabel 2650 2750 0    60   Input ~ 0
@@
 Wire Wire Line
 	1200 2250 1200 2750
-Text GLabel 8450 3900 3    60   Input ~ 0
+Text GLabel 2050 1250 0    60   Input ~ 0
 ~DISABLE_DYNAMO
 Wire Wire Line
@@
 Wire Wire Line
 	8150 3500 8150 3600
-Wire Wire Line
-	8150 2950 8250 2950
-Wire Wire Line
-	8450 3100 8550 3100
 Wire Wire Line
 	7700 2950 7050 2950
@@
 	9850 2800 9850 2950
 Connection ~ 9850 2950
+Connection ~ 3800 1650
 $Comp
 L maxwell-rescue:R-RESCUE-maxwell R?
-U 1 1 5CAC37BE
-P 8250 3650
-AR Path="/5A1FEBCF/5CAC37BE" Ref="R?"  Part="1"
-AR Path="/5A1FEBCF/5C7831A2/5CAC37BE" Ref="R41"  Part="1"
-F 0 "R41" H 8300 3700 50  0000 L CNN
-F 1 "10k" H 8300 3600 50  0000 L CNN
-F 2 "coddingtonbear:0805_Milling" V 8180 3650 50  0001 C CNN
-F 3 "" H 8250 3650 50  0001 C CNN
-	1    8250 3650
-	1    0    0    -1
-$EndComp
-Wire Wire Line
-	8250 3500 8250 2950
-Connection ~ 8250 2950
-Wire Wire Line
-	8250 2950 8550 2950
-Wire Wire Line
-	8450 3100 8450 3800
-Wire Wire Line
-	8250 3800 8450 3800
-Connection ~ 8450 3800
-Wire Wire Line
-	8450 3800 8450 3900
+U 1 1 5CB048BE
+P 2400 1250
+AR Path="/5A1FEBCF/5CB048BE" Ref="R?"  Part="1"
+AR Path="/5A1FEBCF/5C7831A2/5CB048BE" Ref="R41"  Part="1"
+F 0 "R41" H 2200 1300 50  0000 L CNN
+F 1 "340" H 2200 1200 50  0000 L CNN
+F 2 "coddingtonbear:0805_Milling" V 2330 1250 50  0001 C CNN
+F 3 "" H 2400 1250 50  0001 C CNN
+	1    2400 1250
+	0    1    1    0
+$EndComp
+Wire Wire Line
+	8150 2950 8550 2950
+Wire Wire Line
+	2650 1650 3800 1650
+Wire Wire Line
+	2650 1650 2650 2150
+$Comp
+L custom:TRIAC_AAG U22
+U 1 1 5CB2BD5F
+P 2300 1650
+F 0 "U22" V 2472 1650 50  0000 C CNN
+F 1 "BTA20-700CWRG" V 2563 1650 50  0000 C CNN
+F 2 "Package_TO_SOT_THT:TO-220-3_Vertical" H 2300 1650 50  0001 C CNN
+F 3 "" H 2300 1650 50  0000 C CNN
+	1    2300 1650
+	0    1    1    0
+$EndComp
+Wire Wire Line
+	2550 1650 2650 1650
+Connection ~ 2650 1650
+Wire Wire Line
+	2050 1650 1950 1650
+Wire Wire Line
+	2650 1250 2550 1250
+Wire Wire Line
+	2250 1250 2200 1250
+Wire Wire Line
+	2200 1250 2200 1350
+Connection ~ 2200 1250
+Wire Wire Line
+	2200 1250 2050 1250
+$Comp
+L coddingtonbear:+3V3_C #PWR0194
+U 1 1 5CB414CA
+P 2650 1250
+F 0 "#PWR0194" H 2650 1100 50  0001 C CNN
+F 1 "+3V3_C" H 2665 1423 50  0000 C CNN
+F 2 "" H 2650 1250 50  0001 C CNN
+F 3 "" H 2650 1250 50  0001 C CNN
+	1    2650 1250
+	1    0    0    -1
+$EndComp
 $EndSCHEMATC

Commit message: Maxwell Remote v1.9.5
SSRs and Triacs each have voltage drops that are a significant
fraction of how much voltage I have available; let's just use
a latching relay instead.

* Adds Latching relay (and bypass jumper) for allowing one to
  switch off/on the dynamo power source.
Parts:
- removed R41: 340, coddingtonbear:0805_Milling, symbol maxwell-rescue:R-RESCUE-maxwell
- removed U22: BTA20-700CWRG, Package_TO_SOT_THT:TO-220-3_Vertical, symbol custom:TRIAC_AAG
- added JP1: Relay Bypass, coddingtonbear:0805_Milling, symbol Device:Jumper_NO_Small
- added K1: TXS2-L-3V, coddingtonbear:Panasonic_TX-S_DPDT, symbol Relay:AZ850-x
Connections:
- net labels added: DYNAMO_SW_1, DYNAMO_SW_2
- net labels removed: ~DISABLE_DYNAMO
- wire segments 84 -> 81
Changed lines of the file:
@@
 Text GLabel 1100 2750 3    60   Output ~ 0
 V_AC-
-Text GLabel 1950 1650 0    60   Input ~ 0
+Text GLabel 1950 1750 0    60   Input ~ 0
 V_AC+
 Text GLabel 2650 2750 0    60   Input ~ 0
@@
 	8150 3150 8150 2950
 Connection ~ 8150 2950
-Text GLabel 1200 2750 3    60   Output ~ 0
-~DISABLE_DYNAMO
-Wire Wire Line
-	1200 2250 1200 2750
-Text GLabel 2050 1250 0    60   Input ~ 0
-~DISABLE_DYNAMO
+Text GLabel 1200 2750 3    60   BiDi ~ 0
+DYNAMO_SW_2
 Wire Wire Line
 	8150 3450 8150 3500
@@
 Connection ~ 9850 2950
 Connection ~ 3800 1650
-$Comp
-L maxwell-rescue:R-RESCUE-maxwell R?
-U 1 1 5CB048BE
-P 2400 1250
-AR Path="/5A1FEBCF/5CB048BE" Ref="R?"  Part="1"
-AR Path="/5A1FEBCF/5C7831A2/5CB048BE" Ref="R41"  Part="1"
-F 0 "R41" H 2200 1300 50  0000 L CNN
-F 1 "340" H 2200 1200 50  0000 L CNN
-F 2 "coddingtonbear:0805_Milling" V 2330 1250 50  0001 C CNN
-F 3 "" H 2400 1250 50  0001 C CNN
-	1    2400 1250
-	0    1    1    0
-$EndComp
 Wire Wire Line
 	8150 2950 8550 2950
@@
 Wire Wire Line
 	2650 1650 2650 2150
-$Comp
-L custom:TRIAC_AAG U22
-U 1 1 5CB2BD5F
-P 2300 1650
-F 0 "U22" V 2472 1650 50  0000 C CNN
-F 1 "BTA20-700CWRG" V 2563 1650 50  0000 C CNN
-F 2 "Package_TO_SOT_THT:TO-220-3_Vertical" H 2300 1650 50  0001 C CNN
-F 3 "" H 2300 1650 50  0000 C CNN
-	1    2300 1650
-	0    1    1    0
-$EndComp
 Wire Wire Line
 	2550 1650 2650 1650
 Connection ~ 2650 1650
-Wire Wire Line
-	2050 1650 1950 1650
-Wire Wire Line
-	2650 1250 2550 1250
-Wire Wire Line
-	2250 1250 2200 1250
-Wire Wire Line
-	2200 1250 2200 1350
-Connection ~ 2200 1250
-Wire Wire Line
-	2200 1250 2050 1250
-$Comp
-L coddingtonbear:+3V3_C #PWR0194
-U 1 1 5CB414CA
-P 2650 1250
-F 0 "#PWR0194" H 2650 1100 50  0001 C CNN
-F 1 "+3V3_C" H 2665 1423 50  0000 C CNN
-F 2 "" H 2650 1250 50  0001 C CNN
-F 3 "" H 2650 1250 50  0001 C CNN
-	1    2650 1250
-	1    0    0    -1
-$EndComp
+$Comp
+L Relay:AZ850-x K1
+U 1 1 5CB4580B
+P 2250 1750
+F 0 "K1" V 1483 1750 50  0000 C CNN
+F 1 "TXS2-L-3V" V 1574 1750 50  0000 C CNN
+F 2 "coddingtonbear:Panasonic_TX-S_DPDT" H 2800 1800 50  0001 C CNN
+F 3 "http://www.azettler.com/pdfs/az850.pdf" H 2050 1750 50  0001 C CNN
+	1    2250 1750
+	0    1    1    0
+$EndComp
+Text GLabel 1200 2250 1    60   BiDi ~ 0
+DYNAMO_SW_1
+Text GLabel 2550 1350 2    60   BiDi ~ 0
+DYNAMO_SW_1
+Text GLabel 1950 1350 0    60   BiDi ~ 0
+DYNAMO_SW_2
+Text GLabel 1900 700  0    60   Input ~ 0
+V_AC+
+$Comp
+L Device:Jumper_NO_Small JP1
+U 1 1 5CB4DD37
+P 2250 700
+F 0 "JP1" H 2250 885 50  0000 C CNN
+F 1 "Relay Bypass" H 2250 794 50  0000 C CNN
+F 2 "coddingtonbear:0805_Milling" H 2250 700 50  0001 C CNN
+F 3 "~" H 2250 700 50  0001 C CNN
+	1    2250 700
+	1    0    0    -1
+$EndComp
+Wire Wire Line
+	2350 700  3800 700
+Wire Wire Line
+	3800 700  3800 1650
+Wire Wire Line
+	1900 700  2150 700
 $EndSCHEMATC
