File: hardware/maxwell-polarity/maxwell-polarity.sch (KiCad schematic (older format))
At the start: 5 parts, among them J1 Battery, J2 Output, SW1 SW_Push, U1 STT3P2UH7

Commit message: Updating hardware files.
Parts:
- added J?: Conn_01x04, symbol Connector:Conn_01x04
- added U?: STM32F103C8Tx, Housings_QFP:LQFP-48_7x7mm_Pitch0.5mm, symbol MCU_ST_STM32:STM32F103C8Tx
- J1: value Battery -> Output
- J2: value Output -> Battery
Changed lines of the file:
@@
 EESchema Schematic File Version 4
+LIBS:maxwell-polarity-cache
 EELAYER 26 0
 EELAYER END
@@
 L Connector:Conn_01x02 J1
 U 1 1 5A373B31
-P 3450 2100
-F 0 "J1" V 3416 1912 50  0000 R CNN
-F 1 "Battery" V 3325 1912 50  0000 R CNN
-F 2 "monostable/CommonPartsLibrary.pretty:JST_XHP-2" H 3450 2100 50  0001 C CNN
-F 3 "~" H 3450 2100 50  0001 C CNN
-	1    3450 2100
+P 1550 900
+F 0 "J1" V 1516 712 50  0000 R CNN
+F 1 "Output" V 1425 712 50  0000 R CNN
+F 2 "monostable/CommonPartsLibrary.pretty:JST_XHP-2" H 1550 900 50  0001 C CNN
+F 3 "~" H 1550 900 50  0001 C CNN
+	1    1550 900
 	0    -1   -1   0
 $EndComp
@@
 L Connector:Conn_01x02 J2
 U 1 1 5A373B83
-P 4700 2100
-F 0 "J2" V 4666 1912 50  0000 R CNN
-F 1 "Output" V 4575 1912 50  0000 R CNN
-F 2 "monostable/CommonPartsLibrary.pretty:JST_XHP-2" H 4700 2100 50  0001 C CNN
-F 3 "~" H 4700 2100 50  0001 C CNN
-	1    4700 2100
+P 2800 900
+F 0 "J2" V 2766 712 50  0000 R CNN
+F 1 "Battery" V 2675 712 50  0000 R CNN
+F 2 "monostable/CommonPartsLibrary.pretty:JST_XHP-2" H 2800 900 50  0001 C CNN
+F 3 "~" H 2800 900 50  0001 C CNN
+	1    2800 900
 	0    -1   -1   0
 $EndComp
@@
 L coddingtonbear:STT3P2UH7 U1
 U 1 1 5A373FFB
-P 4050 2950
-F 0 "U1" H 4050 2513 60  0000 C CNN
-F 1 "STT3P2UH7" H 4050 2619 60  0000 C CNN
-F 2 "freetronics/freetronics_kicad_library/freetronics_footprints.pretty:SOT23-6" H 4050 2950 60  0001 C CNN
-F 3 "" H 4050 2950 60  0001 C CNN
-	1    4050 2950
+P 2150 1750
+F 0 "U1" H 2150 1313 60  0000 C CNN
+F 1 "STT3P2UH7" H 2150 1419 60  0000 C CNN
+F 2 "freetronics/freetronics_kicad_library/freetronics_footprints.pretty:SOT23-6" H 2150 1750 60  0001 C CNN
+F 3 "" H 2150 1750 60  0001 C CNN
+	1    2150 1750
 	-1   0    0    1
 $EndComp
 Wire Wire Line
-	3550 2300 3550 2700
+	1650 1800 1700 1800
 Wire Wire Line
-	3550 3000 3600 3000
+	2600 1600 2900 1600
 Wire Wire Line
-	4500 2800 4800 2800
+	2900 1600 2900 1100
 Wire Wire Line
-	4800 2800 4800 2300
+	2600 1700 2900 1700
 Wire Wire Line
-	4500 2900 4800 2900
+	2900 1700 2900 1600
+Connection ~ 2900 1600
 Wire Wire Line
-	4800 2900 4800 2800
-Connection ~ 4800 2800
+	2600 1800 2900 1800
 Wire Wire Line
-	4500 3000 4800 3000
+	2900 1800 2900 1700
+Connection ~ 2900 1700
 Wire Wire Line
-	4800 3000 4800 2900
-Connection ~ 4800 2900
+	2600 1900 2900 1900
 Wire Wire Line
-	4500 3100 4800 3100
-Wire Wire Line
-	4800 3100 4800 3000
-Connection ~ 4800 3000
+	2900 1900 2900 1800
+Connection ~ 2900 1800
 $Comp
 L power:GND #PWR01
 U 1 1 5A374253
-P 3050 3700
-F 0 "#PWR01" H 3050 3450 50  0001 C CNN
-F 1 "GND" H 3055 3527 50  0000 C CNN
-F 2 "" H 3050 3700 50  0001 C CNN
-F 3 "" H 3050 3700 50  0001 C CNN
-	1    3050 3700
+P 1150 2500
+F 0 "#PWR01" H 1150 2250 50  0001 C CNN
+F 1 "GND" H 1155 2327 50  0000 C CNN
+F 2 "" H 1150 2500 50  0001 C CNN
+F 3 "" H 1150 2500 50  0001 C CNN
+	1    1150 2500
 	1    0    0    -1
 $EndComp
 Wire Wire Line
-	3450 2450 3450 2350
+	1550 1250 1550 1150
 Wire Wire Line
-	3450 2350 4700 2350
+	1550 1150 2800 1150
 Wire Wire Line
-	4700 2350 4700 2300
-Connection ~ 3450 2350
+	2800 1150 2800 1100
+Connection ~ 1550 1150
 Wire Wire Line
-	3450 2350 3450 2300
+	1550 1150 1550 1100
 $Comp
 L Switch:SW_Push SW1
 U 1 1 5A3744CC
-P 3250 2900
-F 0 "SW1" V 3296 2852 50  0000 R CNN
-F 1 "SW_Push" V 3205 2852 50  0000 R CNN
-F 2 "coddingtonbear/coddingtonbear.pretty:SMD_RED_TACTILE_SWITCH" H 3250 3100 50  0001 C CNN
-F 3 "" H 3250 3100 50  0001 C CNN
-	1    3250 2900
-	0    -1   -1   0
+P 2050 2250
+F 0 "SW1" V 2096 2202 50  0000 R CNN
+F 1 "SW_Push" V 2005 2202 50  0000 R CNN
+F 2 "coddingtonbear/coddingtonbear.pretty:SMD_RED_TACTILE_SWITCH" H 2050 2450 50  0001 C CNN
+F 3 "" H 2050 2450 50  0001 C CNN
+	1    2050 2250
+	1    0    0    -1
 $EndComp
 $Comp
 L device:R R1
 U 1 1 5A3745EC
-P 3200 3450
-F 0 "R1" V 2993 3450 50  0000 C CNN
-F 1 "100k" V 3084 3450 50  0000 C CNN
-F 2 "coddingtonbear/coddingtonbear.pretty:0805_Milling" V 3130 3450 50  0001 C CNN
-F 3 "" H 3200 3450 50  0001 C CNN
-	1    3200 3450
+P 1300 2250
+F 0 "R1" V 1093 2250 50  0000 C CNN
+F 1 "100k" V 1184 2250 50  0000 C CNN
+F 2 "coddingtonbear/coddingtonbear.pretty:0805_Milling" V 1230 2250 50  0001 C CNN
+F 3 "" H 1300 2250 50  0001 C CNN
+	1    1300 2250
 	0    1    1    0
 $EndComp
 Wire Wire Line
-	3050 3450 3050 3700
+	1150 2250 1150 2500
 Wire Wire Line
-	3350 3450 3550 3450
+	1450 2250 1650 2250
 Wire Wire Line
-	3550 3450 3550 3100
+	1650 2250 1650 1900
 Wire Wire Line
-	3550 3100 3600 3100
-Connection ~ 3550 3100
+	1650 1900 1700 1900
 Wire Wire Line
-	3250 3100 3550 3100
+	1550 1250 1150 1250
 Wire Wire Line
-	3250 2700 3550 2700
-Connection ~ 3550 2700
+	1150 1250 1150 2250
+Connection ~ 1150 2250
 Wire Wire Line
-	3550 2700 3550 3000
+	1650 1100 1650 1800
 Wire Wire Line
-	3450 2450 3050 2450
+	1850 2250 1650 2250
+Connection ~ 1650 2250
 Wire Wire Line
-	3050 2450 3050 3450
-Connection ~ 3050 3450
+	2250 2250 2900 2250
+Wire Wire Line
+	2900 2250 2900 1900
+Connection ~ 2900 1900
+$Comp
+L MCU_ST_STM32:STM32F103C8Tx U?
+U 1 1 5A76A5A2
+P 7750 2750
+F 0 "U?" H 7750 4728 50  0000 C CNN
+F 1 "STM32F103C8Tx" H 7750 4637 50  0000 C CNN
+F 2 "Housings_QFP:LQFP-48_7x7mm_Pitch0.5mm" H 10550 4425 50  0001 R TNN
+F 3 "http://www.st.com/st-web-ui/static/active/en/resource/technical/document/datasheet/CD00161566.pdf" H 7750 2750 50  0001 C CNN
+	1    7750 2750
+	1    0    0    -1
+$EndComp
+$Comp
+L Connector:Conn_01x04 J?
+U 1 1 5A76A704
+P 1150 3200
+F 0 "J?" H 1070 2775 50  0000 C CNN
+F 1 "Conn_01x04" H 1070 2866 50  0000 C CNN
+F 2 "" H 1150 3200 50  0001 C CNN
+F 3 "~" H 1150 3200 50  0001 C CNN
+	1    1150 3200
+	-1   0    0    1
+$EndComp
 $EndSCHEMATC

Commit message: Updating maxwell-polarity, but I'm not likely to use those changes; instead, let's just fix maxwel.
Parts:
- removed J1: Output, monostable/CommonPartsLibrary.pretty:JST_XHP-2, symbol Connector:Conn_01x02
- removed J2: Battery, monostable/CommonPartsLibrary.pretty:JST_XHP-2, symbol Connector:Conn_01x02
- removed J?: Conn_01x04, symbol Connector:Conn_01x04
- removed R1: 100k, coddingtonbear/coddingtonbear.pretty:0805_Milling, symbol device:R
- removed SW1: SW_Push, coddingtonbear/coddingtonbear.pretty:SMD_RED_TACTILE_SWITCH, symbol Switch:SW_Push
- removed U1: STT3P2UH7, freetronics/freetronics_kicad_library/freetronics_footprints.pretty:SOT23-6, symbol coddingtonbear:STT3P2UH7
- removed U?: STM32F103C8Tx, Housings_QFP:LQFP-48_7x7mm_Pitch0.5mm, symbol MCU_ST_STM32:STM32F103C8Tx
- added BT?: Battery_Cell, symbol device:Battery_Cell
- added C? (x2): 1u, symbol device:CP
- added C?: 2.2u, symbol device:CP
- added C? (x2): 0.1u, symbol device:C
- added J?: INPUT, symbol Connector:Conn_01x05
- added Q?: NDS332P, symbol device:Q_PMOS_GSD
- added R? (x3): 10k, symbol device:R
- added R?: 60k, symbol device:R
- added R?: 100k, symbol device:R
- added R? (x2): 330, symbol device:R
- added U?: MIC5209-ADJ, symbol coddingtonbear:MIC5209-ADJ
- added U?: SN65HVD235, Housings_SOIC:SOIC-8_3.9x4.9mm_Pitch1.27mm, symbol interface:SN65HVD235
- added U?: ESP-12E, RF_Modules:ESP-12E, symbol rfcom:ESP-12E
- added U?: FGPMMOPA6H, symbol coddingtonbear-gps:FGPMMOPA6H
- added U?: SIM800L_5-pin, symbol coddingtonbear:SIM800L_5-pin
- added U?: ITEAD_HC-05, symbol itead:ITEAD_HC-05
Connections:
- net labels added: +3V3, +BACKUP, +BATT, BOOT0, BT_IN, BT_KEY, BT_OUT, CAN+, CAN-, CAN_RX, CAN_TX, CELLULAR_IN, CELLULAR_OUT, CELLULAR_RST, GPS_IN, GPS_OUT, GPS_RST, WAKE
- wire segments 23 -> 64
Other:
- note added: "* Cellular Radio\n* GPS Module\n* ? WIFI\n* ? Bluetooth"
