File: hardware/maxwell-remote/maxwell-remote.sch (KiCad schematic (older format))
At the start: 44 parts, among them J1 INPUT, J2 UART, J3 Left, J4 Right, J5 Programmer, J6 B0_JMP, J7 B1_JMP, Q2 NDS332P, Q3 NDS332P, Q4 NDS332P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

Commit message: Maxwell-remote v3; swapping HC-05 for ESP32 because all of my HC-05s are dead.
Parts:
- removed J2: UART, coddingtonbear/coddingtonbear.pretty:JST_EH_B02B-EH-A_02x2.50mm_Straight_LargePads, symbol Connector:Conn_01x02
- removed Q3: NDS332P, cvra/kicad-lib/footprints/_std.pretty:SSOT-3, symbol device:Q_PMOS_GSD
- removed R13: 10k, coddingtonbear/coddingtonbear.pretty:0805_Milling, symbol device:R
- removed U7: ITEAD_HC-05, pelrun/libKiCad/footprint/w_rf_modules.pretty:ITEAD_HC-05, symbol W_RTX:ITEAD_HC-05
- added C12: 0.1, coddingtonbear/coddingtonbear.pretty:0805_Milling, symbol device:C
- added J2: UART, coddingtonbear:JST_XH_B03B-XH-A_03x2.50mm_Straight_LargePads, symbol Connector:Conn_01x03
- added J8: SPI2, coddingtonbear:JST_XH_B07B-XH-A_07x2.50mm_Straight_LargePads, symbol Connector:Conn_01x07
- added U2: ESP32-WROOM, OLIMEX/KiCAD/KiCAD_Footprints/OLIMEX_Cases-FP.pretty:ESP-WROOM-32_MODULE, symbol esp32:ESP32-WROOM
- C5: footprint usagi1975/kicad_mod.pretty:Capacitor_Electrolytic_D5.0xP2.0 -> celeritous/KiCad.pretty:CAPACITOR_TANTALUM_B
- C6: footprint usagi1975/kicad_mod.pretty:Capacitor_Electrolytic_D5.0xP2.0 -> celeritous/KiCad.pretty:CAPACITOR_TANTALUM_C
- R7: value 10k -> 330
- U8: footprint coddingtonbear/coddingtonbear.pretty:128x64_OLED_LCD -> coddingtonbear:JST_XH_B04B-XH-A_04x2.50mm_Straight_LargePads
- Y1: footprint brunoeagle/kicad-open-modules:CRYSTAL_SMD -> coddingtonbear/coddingtonbear.pretty:ASFL1
- Y2: footprint KiCad/Crystals.pretty:Crystal_SMD_SeikoEpson_MC306-4pin_8.0x3.2mm -> coddingtonbear:SM-CRYSTAL-ABS25_LargePads
Connections:
- net labels added: BT_IN, BT_OUT, DISBABLE_BLUETOOTH_, SPI_CS_A, SPI_CS_B
- net labels removed: DISBABLE_BLUETOOTH, RX, TX
- wire segments 147 -> 149

Commit message: Fixing problems on maxwell-remote board; adding I2C pull-up resistors; fixing 8Mhz xtal package (required removing 32khz crystal).
Parts:
- removed C3, C4: 22p, coddingtonbear/coddingtonbear.pretty:0805_Milling, symbol device:C
- removed Y2: Crystal_GND23_Small, coddingtonbear:SM-CRYSTAL-ABS25_LargePads, symbol device:Crystal_GND23_Small
- added R13, R17: 2.2k, coddingtonbear/coddingtonbear.pretty:0805_Milling, symbol device:R
- J1: footprint coddingtonbear/coddingtonbear.pretty:JST_EH_B05B-EH-A_05x2.50mm_Straight_LargePads -> coddingtonbear:JST_XH_B05B-XH-A_05x2.50mm_Straight_LargePads
- J3, J4: footprint coddingtonbear/coddingtonbear.pretty:JST_EH_B03B-EH-A_03x2.50mm_Straight_LargePads -> coddingtonbear:JST_XH_B03B-XH-A_03x2.50mm_Straight_LargePads
- Y1: footprint coddingtonbear/coddingtonbear.pretty:ASFL1 -> cpavlina/kicad-pcblib/smd-non-ipc.pretty:Abracon-ABM2
Connections:
- wire segments 149 -> 147
Changed lines of the file:
@@
 F 0 "J1" H 970 675 50  0000 C CNN
 F 1 "INPUT" H 970 766 50  0000 C CNN
-F 2 "coddingtonbear/coddingtonbear.pretty:JST_EH_B05B-EH-A_05x2.50mm_Straight_LargePads" H 1050 1100 50  0001 C CNN
+F 2 "coddingtonbear:JST_XH_B05B-XH-A_05x2.50mm_Straight_LargePads" H 1050 1100 50  0001 C CNN
 F 3 "~" H 1050 1100 50  0001 C CNN
 	1    1050 1100
@@
 	4750 1950 4750 1600
 Connection ~ 4600 1950
-Text GLabel 10050 1450 3    60   BiDi ~ 0
+Text GLabel 10050 1600 3    60   BiDi ~ 0
 SCL
-Text GLabel 10150 1450 3    60   BiDi ~ 0
+Text GLabel 10450 1600 3    60   BiDi ~ 0
 SDA
 Wire Wire Line
@@
 F 0 "J3" V 8316 812 50  0000 R CNN
 F 1 "Left" V 8225 812 50  0000 R CNN
-F 2 "coddingtonbear/coddingtonbear.pretty:JST_EH_B03B-EH-A_03x2.50mm_Straight_LargePads" H 8350 1000 50  0001 C CNN
+F 2 "coddingtonbear:JST_XH_B03B-XH-A_03x2.50mm_Straight_LargePads" H 8350 1000 50  0001 C CNN
 F 3 "~" H 8350 1000 50  0001 C CNN
 	1    8350 1000
@@
 F 0 "J4" V 9116 812 50  0000 R CNN
 F 1 "Right" V 9025 812 50  0000 R CNN
-F 2 "coddingtonbear/coddingtonbear.pretty:JST_EH_B03B-EH-A_03x2.50mm_Straight_LargePads" H 9150 1000 50  0001 C CNN
+F 2 "coddingtonbear:JST_XH_B03B-XH-A_03x2.50mm_Straight_LargePads" H 9150 1000 50  0001 C CNN
 F 3 "~" H 9150 1000 50  0001 C CNN
 	1    9150 1000
@@
 F 0 "Y1" V 1404 4081 50  0000 L CNN
 F 1 "Crystal" V 1495 4081 50  0000 L CNN
-F 2 "coddingtonbear/coddingtonbear.pretty:ASFL1" H 1450 3950 50  0001 C CNN
+F 2 "cpavlina/kicad-pcblib/smd-non-ipc.pretty:Abracon-ABM2" H 1450 3950 50  0001 C CNN
 F 3 "" H 1450 3950 50  0001 C CNN
 	1    1450 3950
@@
 	2200 7150 2200 7500
 Wire Wire Line
-	10050 1350 10050 1450
-Wire Wire Line
 	10150 1450 10150 1350
 $Comp
@@
 	1100 3800 1100 4100
 Connection ~ 1100 4100
-$Comp
-L device:Crystal_GND23_Small Y2
-U 1 1 5ABD0940
-P 1350 4450
-F 0 "Y2" V 1304 4616 50  0000 L CNN
-F 1 "Crystal_GND23_Small" V 1395 4616 50  0000 L CNN
-F 2 "coddingtonbear:SM-CRYSTAL-ABS25_LargePads" H 1350 4450 50  0001 C CNN
-F 3 "" H 1350 4450 50  0001 C CNN
-	1    1350 4450
-	0    1    1    0
-$EndComp
-$Comp
-L device:C C4
-U 1 1 5ABD0A3F
-P 1050 4550
-F 0 "C4" V 798 4550 50  0000 C CNN
-F 1 "22p" V 889 4550 50  0000 C CNN
-F 2 "coddingtonbear/coddingtonbear.pretty:0805_Milling" H 1088 4400 50  0001 C CNN
-F 3 "" H 1050 4550 50  0001 C CNN
-	1    1050 4550
-	0    1    1    0
-$EndComp
-$Comp
-L device:C C3
-U 1 1 5ABD0AAC
-P 1050 4350
-F 0 "C3" V 798 4350 50  0000 C CNN
-F 1 "22p" V 889 4350 50  0000 C CNN
-F 2 "coddingtonbear/coddingtonbear.pretty:0805_Milling" H 1088 4200 50  0001 C CNN
-F 3 "" H 1050 4350 50  0001 C CNN
-	1    1050 4350
-	0    1    1    0
-$EndComp
-Wire Wire Line
-	1700 4300 1350 4300
-Wire Wire Line
-	1350 4300 1350 4350
-Wire Wire Line
-	1700 4400 1500 4400
-Wire Wire Line
-	1500 4400 1500 4550
-Wire Wire Line
-	1500 4550 1350 4550
-Wire Wire Line
-	1350 4550 1200 4550
-Connection ~ 1350 4550
-Wire Wire Line
-	1200 4350 1200 4300
-Wire Wire Line
-	1200 4300 1350 4300
-Connection ~ 1350 4300
-Wire Wire Line
-	900  4550 900  4350
-Wire Wire Line
-	900  4350 900  4100
-Connection ~ 900  4350
-Connection ~ 900  4100
 Wire Wire Line
 	900  4100 1100 4100
@@
 	1    0    0    -1
 $EndComp
+$Comp
+L device:R R13
+U 1 1 5AD2D96A
+P 10150 1750
+F 0 "R13" H 10080 1704 50  0000 R CNN
+F 1 "2.2k" H 10080 1795 50  0000 R CNN
+F 2 "coddingtonbear/coddingtonbear.pretty:0805_Milling" V 10080 1750 50  0001 C CNN
+F 3 "" H 10150 1750 50  0001 C CNN
+	1    10150 1750
+	-1   0    0    1
+$EndComp
+$Comp
+L device:R R17
+U 1 1 5AD2D9E4
+P 10550 1750
+F 0 "R17" H 10480 1704 50  0000 R CNN
+F 1 "2.2k" H 10480 1795 50  0000 R CNN
+F 2 "coddingtonbear/coddingtonbear.pretty:0805_Milling" V 10480 1750 50  0001 C CNN
+F 3 "" H 10550 1750 50  0001 C CNN
+	1    10550 1750
+	-1   0    0    1
+$EndComp
+Wire Wire Line
+	10050 1350 10050 1500
+Wire Wire Line
+	10150 1450 10450 1450
+Wire Wire Line
+	10450 1450 10450 1600
+Wire Wire Line
+	10450 1450 10550 1450
+Wire Wire Line
+	10550 1450 10550 1600
+Connection ~ 10450 1450
+Wire Wire Line
+	10150 1600 10150 1500
+Wire Wire Line
+	10150 1500 10050 1500
+Connection ~ 10050 1500
+Wire Wire Line
+	10050 1500 10050 1600
+$Comp
+L power:+3V3 #PWR030
+U 1 1 5AD557AF
+P 10150 1900
+F 0 "#PWR030" H 10150 1750 50  0001 C CNN
+F 1 "+3V3" H 10165 2073 50  0000 C CNN
+F 2 "" H 10150 1900 50  0001 C CNN
+F 3 "" H 10150 1900 50  0001 C CNN
+	1    10150 1900
+	-1   0    0    1
+$EndComp
+Wire Wire Line
+	10150 1900 10550 1900
+Connection ~ 10150 1900
 $EndSCHEMATC

Commit message: Never made the new version of maxwell remote; reverting schematics to v2.0.
Parts:
- removed C12: 0.1, coddingtonbear/coddingtonbear.pretty:0805_Milling, symbol device:C
- removed J2: UART, coddingtonbear:JST_XH_B03B-XH-A_03x2.50mm_Straight_LargePads, symbol Connector:Conn_01x03
- removed J8: SPI2, coddingtonbear:JST_XH_B07B-XH-A_07x2.50mm_Straight_LargePads, symbol Connector:Conn_01x07
- removed R17: 2.2k, coddingtonbear/coddingtonbear.pretty:0805_Milling, symbol device:R
- removed U2: ESP32-WROOM, OLIMEX/KiCAD/KiCAD_Footprints/OLIMEX_Cases-FP.pretty:ESP-WROOM-32_MODULE, symbol esp32:ESP32-WROOM
- added C3, C4: 22p, coddingtonbear/coddingtonbear.pretty:0805_Milling, symbol device:C
- added J2: UART, coddingtonbear/coddingtonbear.pretty:JST_EH_B02B-EH-A_02x2.50mm_Straight_LargePads, symbol Connector:Conn_01x02
- added Q3: NDS332P, cvra/kicad-lib/footprints/_std.pretty:SSOT-3, symbol device:Q_PMOS_GSD
- added U7: ITEAD_HC-05, pelrun/libKiCad/footprint/w_rf_modules.pretty:ITEAD_HC-05, symbol W_RTX:ITEAD_HC-05
- added Y2: Crystal_GND23_Small, KiCad/Crystals.pretty:Crystal_SMD_SeikoEpson_MC306-4pin_8.0x3.2mm, symbol device:Crystal_GND23_Small
- C5: footprint celeritous/KiCad.pretty:CAPACITOR_TANTALUM_B -> usagi1975/kicad_mod.pretty:Capacitor_Electrolytic_D5.0xP2.0
- C6: footprint celeritous/KiCad.pretty:CAPACITOR_TANTALUM_C -> usagi1975/kicad_mod.pretty:Capacitor_Electrolytic_D5.0xP2.0
- J1: footprint coddingtonbear:JST_XH_B05B-XH-A_05x2.50mm_Straight_LargePads -> coddingtonbear/coddingtonbear.pretty:JST_EH_B05B-EH-A_05x2.50mm_Straight_LargePads
- J3, J4: footprint coddingtonbear:JST_XH_B03B-XH-A_03x2.50mm_Straight_LargePads -> coddingtonbear/coddingtonbear.pretty:JST_EH_B03B-EH-A_03x2.50mm_Straight_LargePads
- R13: value 2.2k -> 10k
- R7: value 330 -> 10k
- U8: footprint coddingtonbear:JST_XH_B04B-XH-A_04x2.50mm_Straight_LargePads -> coddingtonbear/coddingtonbear.pretty:128x64_OLED_LCD
- Y1: footprint cpavlina/kicad-pcblib/smd-non-ipc.pretty:Abracon-ABM2 -> brunoeagle/kicad-open-modules:CRYSTAL_SMD
Connections:
- net labels added: DISBABLE_BLUETOOTH, RX, TX
- net labels removed: BT_IN, BT_OUT, DISBABLE_BLUETOOTH_, SPI_CS_A, SPI_CS_B
