File: hardware/maxwell-remote/maxwell-remote.sch (KiCad schematic (older format))
At the start: 7 parts

Commit message: Adding beginnings of remote PCB.
Parts:
- removed U?: MCP2515-E/ST-SOIC, symbol coddingtonbear:MCP2515-E/ST-SOIC
- added C1, C10, C2, C3, C4, C9: 0.1u, coddingtonbear/coddingtonbear.pretty:0805_Milling, symbol device:C
- added C11: 0.1, coddingtonbear/coddingtonbear.pretty:0805_Milling, symbol device:C
- added C5: 1u, celeritous/KiCad.pretty:CAPACITOR_ELECTROLYTIC_4.3MM, symbol device:CP
- added C6: 2.2u, celeritous/KiCad.pretty:CAPACITOR_ELECTROLYTIC_4.3MM, symbol device:CP
- added C7, C8: 22p, coddingtonbear/coddingtonbear.pretty:0805_Milling, symbol device:C
- added J1: INPUT, KiCad/Connectors_JST.pretty:JST_EH_B05B-EH-A_05x2.50mm_Straight, symbol Connector:Conn_01x05
- added J2: Conn_02x03_Odd_Even, KiCad/Pin_Headers.pretty:Pin_Header_Straight_2x03_Pitch2.54mm_SMD, symbol Connector:Conn_02x03_Odd_Even
- added J3: Left, monostable/CommonPartsLibrary.pretty:JST_XHP-3, symbol Connector:Conn_01x03
- added J4: Right, monostable/CommonPartsLibrary.pretty:JST_XHP-3, symbol Connector:Conn_01x03
- added Q1, Q2, Q3, Q4: NDS332P, cuzdaori/KiCad.pretty:SOT23, symbol device:Q_PMOS_GSD
- added R1, R14, R2, R5, R7, R8, R9: 10k, coddingtonbear/coddingtonbear.pretty:0805_Milling, symbol device:R
- added R10: 330, coddingtonbear/coddingtonbear.pretty:0805_Milling, symbol device:R
- added R11, R12: NC, coddingtonbear/coddingtonbear.pretty:0805_Milling, symbol device:R
- added R13: 0, coddingtonbear/coddingtonbear.pretty:0805_Milling, symbol device:R
- added R3: 60k, coddingtonbear/coddingtonbear.pretty:0805_Milling, symbol device:R
- added R4: 100k, coddingtonbear/coddingtonbear.pretty:0805_Milling, symbol device:R
- added R6: 120, coddingtonbear/coddingtonbear.pretty:0805_Milling, symbol device:R
- added U3: MIC5209-ADJ, OLIMEX/KiCAD/KiCAD_Footprints/OLIMEX_IC-FP.pretty:SOIC-8_208mil, symbol coddingtonbear:MIC5209-ADJ
- added U4: MCP2515-E_ST-SOIC, Tinkerforge/kicad-libraries:SOIC-18, symbol coddingtonbear:MCP2515-E_ST-SOIC
- added U7: ITEAD_HC-05, pelrun/libKiCad/footprint/w_rf_modules.pretty:ITEAD_HC-05, symbol W_RTX:ITEAD_HC-05
- added Y1: Crystal, monostable/CommonPartsLibrary.pretty:XTAL_HC-49US-16.000MHZ, symbol device:Crystal
- BT1: renamed from BT?; footprint (none) -> ashtonchase/Battery_Holders.pretty:BatteryHolder_CoinCell_Keystone_1027
- U1: renamed from U?; footprint MODULE -> KiCad/TO_SOT_Packages_SMD.pretty:TSOT-23-6_MK06A_HandSoldering
- U2: renamed from U?; footprint TQFP44 -> OLIMEX/KiCAD/KiCAD_Footprints/OLIMEX_IC-FP.pretty:TQFP44
- U5: renamed from U?; footprint Housings_SOIC:SOIC-8_3.9x4.9mm_Pitch1.27mm -> OLIMEX/KiCAD/KiCAD_Footprints/OLIMEX_IC-FP.pretty:SOIC-8_208mil
- U6: renamed from U?; footprint (none) -> rascalmicro/rascalmicro-kicad-footprints.pretty:FGPMMOPA6H
- U8: renamed from U?; footprint (none) -> KiCad/Pin_Headers.pretty:Pin_Header_Straight_1x04_Pitch2.54mm
Connections:
- net labels added: +3V3, +BATT, BACKUP_POWER, BT_KEY, CAN+, CAN-, CAN_CS, CAN_INT, ENABLE_SCREEN, GND, MISO, MOSI, RESET, RX, RX_GPS, SCK, SCL, SDA, TX, TX_GPS, WAKE, ~DISABLE_REGULATOR, ~DISBABLE_BLUETOOTH, ~LEFT_A, ~LEFT_B, ~RIGHT_A, ~RIGHT_B
- wire segments 0 -> 167
Other:
- note removed: "add MIC5209"

Commit message: Adding maxwell remote.
Changed lines of the file:
@@
 Text GLabel 5100 5900 0    60   BiDi ~ 0
 SCK
-Text GLabel 3300 4400 2    60   Output ~ 0
+Text GLabel 3150 5000 2    60   Output ~ 0
 CAN_CS
 Text GLabel 5100 5800 0    60   Input ~ 0
@@
 Text GLabel 3150 5700 2    60   BiDi ~ 0
 SDA
-Text GLabel 3300 4100 2    60   BiDi ~ 0
+Text GLabel 3150 4900 2    60   BiDi ~ 0
 WAKE
-Text GLabel 3300 3800 2    60   Output ~ 0
+Text GLabel 3150 4100 2    60   Output ~ 0
 ~DISABLE_REGULATOR
-Text GLabel 3300 3900 2    60   Input ~ 0
+Text GLabel 3150 4000 2    60   Input ~ 0
 BACKUP_POWER
-Text GLabel 3300 4200 2    60   Input ~ 0
+Text GLabel 3150 5100 2    60   Input ~ 0
 CAN_INT
 Text GLabel 6300 6200 2    60   Output ~ 0
@@
 Text GLabel 9400 2150 0    60   Input ~ 0
 ENABLE_SCREEN
-Text GLabel 3300 4000 2    60   Output ~ 0
+Text GLabel 3150 5800 2    60   Output ~ 0
 ENABLE_SCREEN
 Wire Wire Line
@@
 Text GLabel 6300 3500 3    60   Output ~ 0
 ~RIGHT_B
-Text GLabel 3300 4500 2    60   Input ~ 0
+Text GLabel 3150 4400 2    60   Input ~ 0
 ~LEFT_A
-Text GLabel 3300 4700 2    60   Input ~ 0
+Text GLabel 3150 4500 2    60   Input ~ 0
 ~LEFT_B
-Text GLabel 3300 4800 2    60   Input ~ 0
+Text GLabel 3150 4200 2    60   Input ~ 0
 ~RIGHT_A
-Text GLabel 3300 4900 2    60   Input ~ 0
+Text GLabel 3150 4300 2    60   Input ~ 0
 ~RIGHT_B
 Wire Wire Line

Commit message: Adding final version of remote.
Parts:
- removed BT1: Battery_Cell, ashtonchase/Battery_Holders.pretty:BatteryHolder_CoinCell_Keystone_1027, symbol device:Battery_Cell
- removed J2: Conn_02x03_Odd_Even, KiCad/Pin_Headers.pretty:Pin_Header_Straight_2x03_Pitch2.54mm_SMD, symbol Connector:Conn_02x03_Odd_Even
- removed Q1: NDS332P, cuzdaori/KiCad.pretty:SOT23, symbol device:Q_PMOS_GSD
- removed U1: LTC4412, KiCad/TO_SOT_Packages_SMD.pretty:TSOT-23-6_MK06A_HandSoldering, symbol cvra:LTC4412
- removed U2: ATMEGA1284-AU, OLIMEX/KiCAD/KiCAD_Footprints/OLIMEX_IC-FP.pretty:TQFP44, symbol atmel:ATMEGA1284-AU
- removed U4: MCP2515-E_ST-SOIC, Tinkerforge/kicad-libraries:SOIC-18, symbol coddingtonbear:MCP2515-E_ST-SOIC
- removed U6: FGPMMOPA6H, rascalmicro/rascalmicro-kicad-footprints.pretty:FGPMMOPA6H, symbol FPGMMOPA6H.lib:FGPMMOPA6H
- added J5: Programmer, KiCad/Pin_Headers.pretty:Pin_Header_Straight_1x04_Pitch2.54mm, symbol Connector:Conn_01x04
- added R15, R16: 10k, coddingtonbear/coddingtonbear.pretty:0805_Milling, symbol device:R
- added R17, R18: JMP, coddingtonbear/coddingtonbear.pretty:0805_Milling, symbol device:R
- added U1: STM32F103C8Tx, kicad-castellated-breakouts:QFP48-1.27MM-CASTELLATED, symbol MCU_ST_STM32:STM32F103C8Tx
- added Y2: Crystal_GND23_Small, symbol device:Crystal_GND23_Small
- C1, C2, C3, C4: value 0.1u -> 22p
- C7, C8: value 22p -> 0.1
- C9: value 0.1u -> 0.1
- J3, J4: footprint monostable/CommonPartsLibrary.pretty:JST_XHP-3 -> KiCad/Connectors_JST.pretty:JST_EH_B03B-EH-A_03x2.50mm_Straight
- R1, R5: value 10k -> 100k
- R10: value 330 -> 1M
- R11, R12: value NC -> 330
- R13: value 0 -> 10k
- U8: footprint KiCad/Pin_Headers.pretty:Pin_Header_Straight_1x04_Pitch2.54mm -> coddingtonbear/coddingtonbear.pretty:128x64_OLED_LCD
- Y1: footprint monostable/CommonPartsLibrary.pretty:XTAL_HC-49US-16.000MHZ -> brunoeagle/kicad-open-modules:CRYSTAL_SMD
Connections:
- net labels added: BOOT0, BOOT1, CAN_RX, CAN_TX, SWCLK, SWDIO
- net labels removed: BACKUP_POWER, CAN_CS, CAN_INT, MISO, MOSI, RESET, RX_GPS, SCK, TX_GPS, ~DISABLE_REGULATOR
- wire segments 167 -> 147

Commit message: Updating maxwell-remote to v2.0; adds a variety of fixes including:
Layout:

* Use of incorrect footprint for NDS332 (should be SSOT-3 rathe
  than SOT-23)
* Inverted default powered states for screen and bluetooth module.
* Fixed 32kHz crystal footprint.
* Swapped surface-mount capacitors for through-hole for durability.
  I've torn the surface-mount ones off the board at least twice now;
  they are not likely to survive long in a high-vibration environment.
* General layout improvements.

Functional:

* Linked both UART2 and UART1 to Bluetooth module.  Only UART1 can be
  used for programming, but UART1 is _usually_ used for SerialUSB and
  thus should be avoided given that the USB hardware shares memory with
  the CAN hardware.
* Added a RX/TX JST connector.  This is partially to improve my ability
  to solder to the fcu layer (by adding an additional plastic support to
  the underside of the board), but also because it does make it easier
  to troubleshoot.
Parts:
- added J2: UART, KiCad/Connectors_JST.pretty:JST_PH_B2B-PH-K_02x2.00mm_Straight, symbol Connector:Conn_01x02
- C5, C6: footprint celeritous/KiCad.pretty:CAPACITOR_ELECTROLYTIC_4.3MM -> usagi1975/kicad_mod.pretty:Capacitor_Electrolytic_D5.0xP2.0
- Q2, Q3, Q4: footprint cuzdaori/KiCad.pretty:SOT23 -> cvra/kicad-lib/footprints/_std.pretty:SSOT-3
- Y2: footprint (none) -> KiCad/Crystals.pretty:Crystal_SMD_SeikoEpson_MC306-4pin_8.0x3.2mm
Changed lines of the file:
@@
 F 0 "C5" H 3968 1746 50  0000 L CNN
 F 1 "1u" H 3968 1655 50  0000 L CNN
-F 2 "celeritous/KiCad.pretty:CAPACITOR_ELECTROLYTIC_4.3MM" H 3888 1550 50  0001 C CNN
+F 2 "usagi1975/kicad_mod.pretty:Capacitor_Electrolytic_D5.0xP2.0" H 3888 1550 50  0001 C CNN
 F 3 "" H 3850 1700 50  0001 C CNN
 	1    3850 1700
@@
 F 0 "C6" H 4418 1796 50  0000 L CNN
 F 1 "2.2u" H 4418 1705 50  0000 L CNN
-F 2 "celeritous/KiCad.pretty:CAPACITOR_ELECTROLYTIC_4.3MM" H 4338 1600 50  0001 C CNN
+F 2 "usagi1975/kicad_mod.pretty:Capacitor_Electrolytic_D5.0xP2.0" H 4338 1600 50  0001 C CNN
 F 3 "" H 4300 1750 50  0001 C CNN
 	1    4300 1750
@@
 F 0 "Q2" V 3943 1500 50  0000 C CNN
 F 1 "NDS332P" V 3852 1500 50  0000 C CNN
-F 2 "cuzdaori/KiCad.pretty:SOT23" H 3800 1600 50  0001 C CNN
+F 2 "cvra/kicad-lib/footprints/_std.pretty:SSOT-3" H 3800 1600 50  0001 C CNN
 F 3 "" H 3600 1500 50  0001 C CNN
 	1    3600 1500
@@
 Text GLabel 7600 1700 2    60   BiDi ~ 0
 CAN-
-Text GLabel 7500 4900 2    60   BiDi ~ 0
+Text GLabel 7500 5100 2    60   BiDi ~ 0
 WAKE
 $Comp
@@
 F 0 "Q4" H 9956 2196 50  0000 L CNN
 F 1 "NDS332P" H 9956 2105 50  0000 L CNN
-F 2 "cuzdaori/KiCad.pretty:SOT23" H 9950 2250 50  0001 C CNN
+F 2 "cvra/kicad-lib/footprints/_std.pretty:SSOT-3" H 9950 2250 50  0001 C CNN
 F 3 "" H 9750 2150 50  0001 C CNN
 	1    9750 2150
@@
 $EndComp
 Wire Wire Line
-	9850 2350 9850 2600
+	9850 2350 9850 2550
 $Comp
 L device:R R8
@@
 	-1   0    0    1
 $EndComp
-$Comp
-L power:GND #PWR028
-U 1 1 5A44C1CC
-P 9450 2500
-F 0 "#PWR028" H 9450 2250 50  0001 C CNN
-F 1 "GND" H 9455 2327 50  0000 C CNN
-F 2 "" H 9450 2500 50  0001 C CNN
-F 3 "" H 9450 2500 50  0001 C CNN
-	1    9450 2500
-	1    0    0    -1
-$EndComp
 Wire Wire Line
 	9450 2150 9550 2150
-Wire Wire Line
-	9450 2450 9450 2500
 Text GLabel 9400 2150 0    60   Input ~ 0
 ENABLE_SCREEN
@@
 F 0 "Q3" H 9006 3546 50  0000 L CNN
 F 1 "NDS332P" H 9006 3455 50  0000 L CNN
-F 2 "cuzdaori/KiCad.pretty:SOT23" H 9000 3600 50  0001 C CNN
+F 2 "cvra/kicad-lib/footprints/_std.pretty:SSOT-3" H 9000 3600 50  0001 C CNN
 F 3 "" H 8800 3500 50  0001 C CNN
 	1    8800 3500
@@
 	1    0    0    -1
 $EndComp
-Wire Wire Line
-	8600 3600 8150 3600
-Wire Wire Line
-	8250 3300 8150 3300
-Wire Wire Line
-	8150 3300 8150 3600
-Connection ~ 8150 3600
-Wire Wire Line
-	8150 3600 7800 3600
 Wire Wire Line
 	8550 3300 8800 3300
@@
 F 0 "Y2" V 1404 4566 50  0000 L CNN
 F 1 "Crystal_GND23_Small" V 1495 4566 50  0000 L CNN
-F 2 "" H 1450 4400 50  0001 C CNN
+F 2 "KiCad/Crystals.pretty:Crystal_SMD_SeikoEpson_MC306-4pin_8.0x3.2mm" H 1450 4400 50  0001 C CNN
 F 3 "" H 1450 4400 50  0001 C CNN
 	1    1450 4400
@@
 Wire Wire Line
 	1450 4550 1650 4550
+$Comp
+L power:GND #PWR022
+U 1 1 5A742B39
+P 8100 3300
+F 0 "#PWR022" H 8100 3050 50  0001 C CNN
+F 1 "GND" H 8105 3127 50  0000 C CNN
+F 2 "" H 8100 3300 50  0001 C CNN
+F 3 "" H 8100 3300 50  0001 C CNN
+	1    8100 3300
+	1    0    0    -1
+$EndComp
+Wire Wire Line
+	8250 3300 8100 3300
+Wire Wire Line
+	7800 3600 8600 3600
+Wire Wire Line
+	9450 2550 9850 2550
+Wire Wire Line
+	9450 2450 9450 2550
+Connection ~ 9850 2550
+Wire Wire Line
+	9850 2550 9850 2600
+Text GLabel 7500 4800 2    60   Output ~ 0
+TX
+Text GLabel 7500 4900 2    60   Input ~ 0
+RX
+$Comp
+L Connector:Conn_01x02 J2
+U 1 1 5A743381
+P 8400 4750
+F 0 "J2" V 8366 4562 50  0000 R CNN
+F 1 "UART" V 8275 4562 50  0000 R CNN
+F 2 "KiCad/Connectors_JST.pretty:JST_PH_B2B-PH-K_02x2.00mm_Straight" H 8400 4750 50  0001 C CNN
+F 3 "~" H 8400 4750 50  0001 C CNN
+	1    8400 4750
+	0    -1   -1   0
+$EndComp
+Text GLabel 8400 4950 3    60   Output ~ 0
+TX
+Text GLabel 8500 4950 3    60   Input ~ 0
+RX
 $EndSCHEMATC

Commit message: Better mini unpopulated boot jumper footprint
Parts:
- removed R17, R18: JMP, coddingtonbear/coddingtonbear.pretty:0805_Milling, symbol device:R
- added J6: B0_JMP, coddingtonbear/coddingtonbear.pretty:Pin_Header_Straight_1x02_Pitch1.27mm_JMP, symbol Connector:Conn_01x02
- added J7: B1_JMP, coddingtonbear/coddingtonbear.pretty:Pin_Header_Straight_1x02_Pitch1.27mm_JMP, symbol Connector:Conn_01x02
- J1: footprint KiCad/Connectors_JST.pretty:JST_EH_B05B-EH-A_05x2.50mm_Straight -> coddingtonbear/coddingtonbear.pretty:JST_EH_B05B-EH-A_05x2.50mm_Straight_LargePads
- J2: footprint KiCad/Connectors_JST.pretty:JST_PH_B2B-PH-K_02x2.00mm_Straight -> coddingtonbear/coddingtonbear.pretty:JST_EH_B02B-EH-A_02x2.50mm_Straight_LargePads
- J3, J4: footprint KiCad/Connectors_JST.pretty:JST_EH_B03B-EH-A_03x2.50mm_Straight -> coddingtonbear/coddingtonbear.pretty:JST_EH_B03B-EH-A_03x2.50mm_Straight_LargePads
- J5: footprint KiCad/Pin_Headers.pretty:Pin_Header_Straight_1x04_Pitch2.54mm -> coddingtonbear/coddingtonbear.pretty:Pin_Header_Straight_1x04_Pitch2.54mm_LargePads
Connections:
- net labels added: DISBABLE_BLUETOOTH, ~ENABLE_SCREEN
- net labels removed: ENABLE_SCREEN, ~DISBABLE_BLUETOOTH
Changed lines of the file:
@@
 F 0 "J1" H 970 675 50  0000 C CNN
 F 1 "INPUT" H 970 766 50  0000 C CNN
-F 2 "KiCad/Connectors_JST.pretty:JST_EH_B05B-EH-A_05x2.50mm_Straight" H 1050 1100 50  0001 C CNN
+F 2 "coddingtonbear/coddingtonbear.pretty:JST_EH_B05B-EH-A_05x2.50mm_Straight_LargePads" H 1050 1100 50  0001 C CNN
 F 3 "~" H 1050 1100 50  0001 C CNN
 	1    1050 1100
@@
 	9450 2150 9550 2150
 Text GLabel 9400 2150 0    60   Input ~ 0
-ENABLE_SCREEN
+~ENABLE_SCREEN
 Text GLabel 1700 5000 0    60   Output ~ 0
-ENABLE_SCREEN
+~ENABLE_SCREEN
 Wire Wire Line
 	9400 2150 9450 2150
@@
 	8550 3300 8800 3300
 Text GLabel 8800 3050 0    60   Input ~ 0
-~DISBABLE_BLUETOOTH
+DISBABLE_BLUETOOTH
 Wire Wire Line
 	8800 3050 8800 3300
@@
 F 0 "J3" V 8316 812 50  0000 R CNN
 F 1 "Left" V 8225 812 50  0000 R CNN
-F 2 "KiCad/Connectors_JST.pretty:JST_EH_B03B-EH-A_03x2.50mm_Straight" H 8350 1000 50  0001 C CNN
+F 2 "coddingtonbear/coddingtonbear.pretty:JST_EH_B03B-EH-A_03x2.50mm_Straight_LargePads" H 8350 1000 50  0001 C CNN
 F 3 "~" H 8350 1000 50  0001 C CNN
 	1    8350 1000
@@
 F 0 "J4" V 9116 812 50  0000 R CNN
 F 1 "Right" V 9025 812 50  0000 R CNN
-F 2 "KiCad/Connectors_JST.pretty:JST_EH_B03B-EH-A_03x2.50mm_Straight" H 9150 1000 50  0001 C CNN
+F 2 "coddingtonbear/coddingtonbear.pretty:JST_EH_B03B-EH-A_03x2.50mm_Straight_LargePads" H 9150 1000 50  0001 C CNN
 F 3 "~" H 9150 1000 50  0001 C CNN
 	1    9150 1000
@@
 $EndComp
 Text GLabel 1700 5700 0    60   Output ~ 0
-~DISBABLE_BLUETOOTH
+DISBABLE_BLUETOOTH
 Text GLabel 6500 1500 0    60   Input ~ 0
 CAN_TX
@@
 F 0 "J5" H 5980 6942 50  0000 L CNN
 F 1 "Programmer" H 5980 6851 50  0000 L CNN
-F 2 "KiCad/Pin_Headers.pretty:Pin_Header_Straight_1x04_Pitch2.54mm" H 5900 6950 50  0001 C CNN
+F 2 "coddingtonbear/coddingtonbear.pretty:Pin_Header_Straight_1x04_Pitch2.54mm_LargePads" H 5900 6950 50  0001 C CNN
 F 3 "~" H 5900 6950 50  0001 C CNN
 	1    5900 6950
@@
 $EndComp
 Wire Wire Line
-	4400 6500 4500 6500
-Wire Wire Line
-	4500 6500 4550 6500
-Connection ~ 4500 6500
-Wire Wire Line
-	4700 6500 4600 6500
-Connection ~ 4600 6500
-Wire Wire Line
 	4550 6600 4550 6500
 Connection ~ 4550 6500
-Wire Wire Line
-	4550 6500 4600 6500
-Text GLabel 2250 7050 2    60   BiDi ~ 0
+Text GLabel 2500 7050 1    60   BiDi ~ 0
 BOOT0
 Text GLabel 1700 3500 0    60   BiDi ~ 0
 BOOT0
-Text GLabel 2250 7200 2    60   BiDi ~ 0
+Text GLabel 2650 7050 1    60   BiDi ~ 0
 BOOT1
 Text GLabel 1700 4800 0    60   BiDi ~ 0
@@
 L device:R R1
 U 1 1 5A6B09A1
-P 2100 7050
-F 0 "R1" H 2030 7004 50  0000 R CNN
-F 1 "100k" H 2030 7095 50  0000 R CNN
-F 2 "coddingtonbear/coddingtonbear.pretty:0805_Milling" V 2030 7050 50  0001 C CNN
-F 3 "" H 2100 7050 50  0001 C CNN
-	1    2100 7050
-	0    1    1    0
+P 2500 7200
+F 0 "R1" H 2430 7154 50  0000 R CNN
+F 1 "100k" H 2430 7245 50  0000 R CNN
+F 2 "coddingtonbear/coddingtonbear.pretty:0805_Milling" V 2430 7200 50  0001 C CNN
+F 3 "" H 2500 7200 50  0001 C CNN
+	1    2500 7200
+	1    0    0    -1
 $EndComp
 $Comp
 L device:R R5
 U 1 1 5A6B0A45
-P 2100 7200
-F 0 "R5" H 2030 7154 50  0000 R CNN
-F 1 "100k" H 2030 7245 50  0000 R CNN
-F 2 "coddingtonbear/coddingtonbear.pretty:0805_Milling" V 2030 7200 50  0001 C CNN
-F 3 "" H 2100 7200 50  0001 C CNN
-	1    2100 7200
-	0    -1   -1   0
+P 2650 7200
+F 0 "R5" H 2580 7154 50  0000 R CNN
+F 1 "100k" H 2580 7245 50  0000 R CNN
+F 2 "coddingtonbear/coddingtonbear.pretty:0805_Milling" V 2580 7200 50  0001 C CNN
+F 3 "" H 2650 7200 50  0001 C CNN
+	1    2650 7200
+	-1   0    0    1
 $EndComp
 $Comp
 L power:GND #PWR011
 U 1 1 5A6B0C29
-P 1950 7200
-F 0 "#PWR011" H 1950 6950 50  0001 C CNN
-F 1 "GND" H 1955 7027 50  0000 C CNN
-F 2 "" H 1950 7200 50  0001 C CNN
-F 3 "" H 1950 7200 50  0001 C CNN
-	1    1950 7200
-	1    0    0    -1
+P 2650 7350
+F 0 "#PWR011" H 2650 7100 50  0001 C CNN
+F 1 "GND" H 2655 7177 50  0000 C CNN
+F 2 "" H 2650 7350 50  0001 C CNN
+F 3 "" H 2650 7350 50  0001 C CNN
+	1    2650 7350
+	0    -1   -1   0
 $EndComp
 $Comp
@@
 Connection ~ 1450 4550
 Wire Wire Line
-	1950 7200 1950 7050
-Connection ~ 1950 7200
-$Comp
-L device:R R17
-U 1 1 5A72F907
-P 2100 6750
-F 0 "R17" H 2030 6704 50  0000 R CNN
-F 1 "JMP" H 2030 6795 50  0000 R CNN
-F 2 "coddingtonbear/coddingtonbear.pretty:0805_Milling" V 2030 6750 50  0001 C CNN
-F 3 "" H 2100 6750 50  0001 C CNN
-	1    2100 6750
-	0    1    1    0
-$EndComp
-$Comp
-L device:R R18
-U 1 1 5A74471B
-P 2100 7550
-F 0 "R18" H 2030 7504 50  0000 R CNN
-F 1 "JMP" H 2030 7595 50  0000 R CNN
-F 2 "coddingtonbear/coddingtonbear.pretty:0805_Milling" V 2030 7550 50  0001 C CNN
-F 3 "" H 2100 7550 50  0001 C CNN
-	1    2100 7550
-	0    1    1    0
-$EndComp
+	2650 7350 2500 7350
+Connection ~ 2650 7350
 $Comp
 L power:+3V3 #PWR012
 U 1 1 5A7447A5
-P 1800 6750
-F 0 "#PWR012" H 1800 6600 50  0001 C CNN
-F 1 "+3V3" H 1815 6923 50  0000 C CNN
-F 2 "" H 1800 6750 50  0001 C CNN
-F 3 "" H 1800 6750 50  0001 C CNN
-	1    1800 6750
-	1    0    0    -1
-$EndComp
-Wire Wire Line
-	1800 6750 1950 6750
-Wire Wire Line
-	2250 6750 2250 7050
-Wire Wire Line
-	2250 7550 2250 7200
-Wire Wire Line
-	1950 7550 1800 7550
-Wire Wire Line
-	1800 7550 1800 6750
-Connection ~ 1800 6750
+P 2200 7500
+F 0 "#PWR012" H 2200 7350 50  0001 C CNN
+F 1 "+3V3" H 2215 7673 50  0000 C CNN
+F 2 "" H 2200 7500 50  0001 C CNN
+F 3 "" H 2200 7500 50  0001 C CNN
+	1    2200 7500
+	0    -1   -1   0
+$EndComp
+Wire Wire Line
+	2200 7050 2500 7050
+Wire Wire Line
+	3000 7050 2650 7050
+Wire Wire Line
+	3000 7500 2200 7500
+Connection ~ 2200 7500
 $Comp
 L device:C C3
@@
 F 0 "J2" V 8366 4562 50  0000 R CNN
 F 1 "UART" V 8275 4562 50  0000 R CNN
-F 2 "KiCad/Connectors_JST.pretty:JST_PH_B2B-PH-K_02x2.00mm_Straight" H 8400 4750 50  0001 C CNN
+F 2 "coddingtonbear/coddingtonbear.pretty:JST_EH_B02B-EH-A_02x2.50mm_Straight_LargePads" H 8400 4750 50  0001 C CNN
 F 3 "~" H 8400 4750 50  0001 C CNN
 	1    8400 4750
@@
 Text GLabel 8500 4950 3    60   Input ~ 0
 RX
+$Comp
+L Connector:Conn_01x02 J7
+U 1 1 5A761DF6
+P 3200 7050
+F 0 "J7" H 3280 7042 50  0000 L CNN
+F 1 "B1_JMP" H 3280 6951 50  0000 L CNN
+F 2 "coddingtonbear/coddingtonbear.pretty:Pin_Header_Straight_1x02_Pitch1.27mm_JMP" H 3200 7050 50  0001 C CNN
+F 3 "~" H 3200 7050 50  0001 C CNN
+	1    3200 7050
+	1    0    0    -1
+$EndComp
+Connection ~ 4600 6500
+Wire Wire Line
+	4550 6500 4600 6500
+Wire Wire Line
+	4700 6500 4600 6500
+Connection ~ 4500 6500
+Wire Wire Line
+	4500 6500 4550 6500
+Wire Wire Line
+	4400 6500 4500 6500
+$Comp
+L Connector:Conn_01x02 J6
+U 1 1 5A77B1E4
+P 2000 7150
+F 0 "J6" H 1920 6825 50  0000 C CNN
+F 1 "B0_JMP" H 1920 6916 50  0000 C CNN
+F 2 "coddingtonbear/coddingtonbear.pretty:Pin_Header_Straight_1x02_Pitch1.27mm_JMP" H 2000 7150 50  0001 C CNN
+F 3 "~" H 2000 7150 50  0001 C CNN
+	1    2000 7150
+	-1   0    0    1
+$EndComp
+Wire Wire Line
+	3000 7150 3000 7500
+Wire Wire Line
+	2200 7150 2200 7500
 $EndSCHEMATC

Commit message: Maxwell-remote v4; just a ton of changes.
Parts:
- removed J2: UART, coddingtonbear/coddingtonbear.pretty:JST_EH_B02B-EH-A_02x2.50mm_Straight_LargePads, symbol Connector:Conn_01x02
- removed Q3: NDS332P, cvra/kicad-lib/footprints/_std.pretty:SSOT-3, symbol device:Q_PMOS_GSD
- removed R11: 330, coddingtonbear/coddingtonbear.pretty:0805_Milling, symbol device:R
- removed U7: ITEAD_HC-05, pelrun/libKiCad/footprint/w_rf_modules.pretty:ITEAD_HC-05, symbol W_RTX:ITEAD_HC-05
- removed Y2: Crystal_GND23_Small, KiCad/Crystals.pretty:Crystal_SMD_SeikoEpson_MC306-4pin_8.0x3.2mm, symbol device:Crystal_GND23_Small
- added C12: 0.1, coddingtonbear/coddingtonbear.pretty:0805_Milling, symbol device:C
- added J2: UART, coddingtonbear:JST_XH_B03B-XH-A_03x2.50mm_Straight_LargePads, symbol Connector:Conn_01x03
- added J8: SPI2, coddingtonbear:JST_XH_B06B-XH-A_06x2.50mm_Straight_LargePads, symbol Connector:Conn_01x06
- added J9: ESP_BM, coddingtonbear/coddingtonbear.pretty:Pin_Header_Straight_1x02_Pitch1.27mm_JMP, symbol Connector:Conn_01x02
- added R17: 2.2k, coddingtonbear/coddingtonbear.pretty:0805_Milling, symbol device:R
- added U2: ESP32-WROOM, OLIMEX/KiCAD/KiCAD_Footprints/OLIMEX_Cases-FP.pretty:ESP-WROOM-32_MODULE, symbol esp32:ESP32-WROOM
- added Y2: Crystal_GND23, coddingtonbear:SM-CRYSTAL-ABS25_LargePads, symbol device:Crystal_GND23
- C5: footprint usagi1975/kicad_mod.pretty:Capacitor_Electrolytic_D5.0xP2.0 -> celeritous/KiCad.pretty:CAPACITOR_TANTALUM_B
- C6: footprint usagi1975/kicad_mod.pretty:Capacitor_Electrolytic_D5.0xP2.0 -> celeritous/KiCad.pretty:CAPACITOR_TANTALUM_C
- J1: footprint coddingtonbear/coddingtonbear.pretty:JST_EH_B05B-EH-A_05x2.50mm_Straight_LargePads -> coddingtonbear:JST_XH_B05B-XH-A_05x2.50mm_Straight_LargePads
- J3, J4: footprint coddingtonbear/coddingtonbear.pretty:JST_EH_B03B-EH-A_03x2.50mm_Straight_LargePads -> coddingtonbear:JST_XH_B03B-XH-A_03x2.50mm_Straight_LargePads
- R12: value 330 -> 10k
- R13: value 10k -> 2.2k
- R7: value 10k -> 330
- U8: footprint coddingtonbear/coddingtonbear.pretty:128x64_OLED_LCD -> coddingtonbear:JST_XH_B04B-XH-A_04x2.50mm_Straight_LargePads
- Y1: footprint brunoeagle/kicad-open-modules:CRYSTAL_SMD -> cpavlina/kicad-pcblib/smd-non-ipc.pretty:Abracon-ABM2
Connections:
- net labels added: BT_IN, BT_OUT, DISBABLE_BLUETOOTH_, ESP_BOOT_MODE, MC_IN, MC_OUT, NRST, SPI_CS
- net labels removed: DISBABLE_BLUETOOTH, RX, TX
- wire segments 147 -> 153
- no-connect marks 0 -> 7
