File: hardware/maxwell-remote/maxwell-remote.sch (KiCad schematic (older format))
At the start: 46 parts, among them J1 INPUT, J2 UART, J3 Left, J4 Right, J5 Programmer, J6 B0_JMP, J7 B1_JMP, J8 SPI2, J9 ESP_BM, Q2 NDS332P, Q4 NDS332P, U1 STM32F103C8Tx, U2 ESP32-WROOM, U3 MIC5209-ADJ, U5 SN65HVD235, U8 OLED-SSD1306, Y1 Crystal, Y2 Crystal_GND23

Commit message: Updating to multi-board linked by FPC connectors.
Parts:
- removed C10: 0.1u, coddingtonbear/coddingtonbear.pretty:0805_Milling, symbol device:C
- removed C5: 1u, celeritous/KiCad.pretty:CAPACITOR_TANTALUM_B, symbol device:CP
- removed C6: 2.2u, celeritous/KiCad.pretty:CAPACITOR_TANTALUM_C, symbol device:CP
- removed J1: INPUT, coddingtonbear:JST_XH_B05B-XH-A_05x2.50mm_Straight_LargePads, symbol Connector:Conn_01x05
- removed J3: Left, coddingtonbear:JST_XH_B03B-XH-A_03x2.50mm_Straight_LargePads, symbol Connector:Conn_01x03
- removed J4: Right, coddingtonbear:JST_XH_B03B-XH-A_03x2.50mm_Straight_LargePads, symbol Connector:Conn_01x03
- removed J8: SPI2, coddingtonbear:JST_XH_B06B-XH-A_06x2.50mm_Straight_LargePads, symbol Connector:Conn_01x06
- removed Q2, Q4: NDS332P, cvra/kicad-lib/footprints/_std.pretty:SSOT-3, symbol device:Q_PMOS_GSD
- removed R13, R17: 2.2k, coddingtonbear/coddingtonbear.pretty:0805_Milling, symbol device:R
- removed R14, R2, R8: 10k, coddingtonbear/coddingtonbear.pretty:0805_Milling, symbol device:R
- removed R3: 60k, coddingtonbear/coddingtonbear.pretty:0805_Milling, symbol device:R
- removed R4: 100k, coddingtonbear/coddingtonbear.pretty:0805_Milling, symbol device:R
- removed R6: 120, coddingtonbear/coddingtonbear.pretty:0805_Milling, symbol device:R
- removed U2: ESP32-WROOM, OLIMEX/KiCAD/KiCAD_Footprints/OLIMEX_Cases-FP.pretty:ESP-WROOM-32_MODULE, symbol esp32:ESP32-WROOM
- removed U3: MIC5209-ADJ, OLIMEX/KiCAD/KiCAD_Footprints/OLIMEX_IC-FP.pretty:SOIC-8_208mil, symbol coddingtonbear:MIC5209-ADJ
- removed U5: SN65HVD235, OLIMEX/KiCAD/KiCAD_Footprints/OLIMEX_IC-FP.pretty:SOIC-8_208mil, symbol interface:SN65HVD235
- removed U8: OLED-SSD1306, coddingtonbear:JST_XH_B04B-XH-A_04x2.50mm_Straight_LargePads, symbol coddingtonbear:OLED-SSD1306
- added J3: FPC 1, coddingtonbear/coddingtonbear.pretty:10P_FPC_1.0mm, symbol Connector:Conn_01x10
- added J4: FPC 2, coddingtonbear/coddingtonbear.pretty:10P_FPC_1.0mm, symbol Connector:Conn_01x10
- added U2: ESP32-WROOM, NorbotNorway/NorBotKiCadFootprints.pretty:ESP32-WROOM, symbol esp32-local:ESP32-WROOM
Connections:
- net labels added: SCREEN_A0, SPI1_MISO, SPI1_MOSI, SPI1_SCK, ~ENABLE_SCREEN_BACKLIGHT, ~SCREEN_CS, ~SCREEN_RST, ~SPI1_CS_2, ~SPI1_CS_3, ~SPI1_CS_4
- net labels removed: +BATT, CAN+, CAN-, SCL, SDA, SPI_CS
- wire segments 153 -> 80
