File: hardware/maxwell-remote/maxwell-remote.sch (KiCad schematic (older format))
At the start: 28 parts, among them J2 UART, J3 FPC 1, J4 FPC 2, J5 Programmer, J6 B0_JMP, J7 B1_JMP, J9 ESP_BM, U1 STM32F103C8Tx, U2 ESP32-WROOM, Y1 Crystal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

Commit message: Updating to v5.0 of the remote's main PCB.
Changed lines of the file:
@@
 	1    0    0    -1
 $EndComp
-Text GLabel 7500 5800 2    60   Output ~ 0
+Text GLabel 7500 4800 2    60   Output ~ 0
 DISBABLE_BLUETOOTH_
 Text GLabel 7850 1400 0    60   Input ~ 0
@@
 L device:R R7
 U 1 1 5AAEE024
-P 8950 4950
-F 0 "R7" H 8880 4904 50  0000 R CNN
-F 1 "330" H 8880 4995 50  0000 R CNN
-F 2 "coddingtonbear/coddingtonbear.pretty:0805_Milling" V 8880 4950 50  0001 C CNN
-F 3 "" H 8950 4950 50  0001 C CNN
-	1    8950 4950
+P 11100 4900
+F 0 "R7" H 11030 4854 50  0000 R CNN
+F 1 "330" H 11030 4945 50  0000 R CNN
+F 2 "coddingtonbear/coddingtonbear.pretty:0805_Milling" V 11030 4900 50  0001 C CNN
+F 3 "" H 11100 4900 50  0001 C CNN
+	1    11100 4900
 	0    -1   -1   0
 $EndComp
-Text GLabel 8800 4950 0    60   BiDi ~ 0
+Text GLabel 11250 4900 2    60   BiDi ~ 0
 BOOT0
 $Comp
@@
 Text GLabel 1650 3300 1    60   Input ~ 0
 NRST
-Text GLabel 10950 3900 2    60   Output ~ 0
+Text GLabel 9100 4450 0    60   Output ~ 0
 NRST
 NoConn ~ 9800 5600
@@
 NoConn ~ 10200 5600
 NoConn ~ 10300 5600
-Text GLabel 9700 5600 3    60   Input ~ 0
+Text GLabel 9100 4350 0    60   Input ~ 0
 BT_KEY
-Text GLabel 7500 5700 2    60   Output ~ 0
+Text GLabel 7500 4700 2    60   Output ~ 0
 BT_KEY
 NoConn ~ 9100 5150
-Text GLabel 10950 5000 2    60   Input ~ 0
-ESP_BOOT_MODE
-Text GLabel 7500 4900 2    60   Output ~ 0
-ESP_BOOT_MODE
 $Comp
 L Connector:Conn_01x02 J9
@@
 	-1   0    0    1
 $EndComp
-Text GLabel 7500 5400 2    60   Output ~ 0
+Text GLabel 1700 5800 0    60   Output ~ 0
 ~ENABLE_SCREEN
 Text GLabel 9950 1200 0    60   Input ~ 0
@@
 Text GLabel 9950 1500 0    60   Input ~ 0
 ~SCREEN_CS
-Text GLabel 1700 5900 0    60   Output ~ 0
+Text GLabel 1700 6100 0    60   Output ~ 0
 ~SCREEN_CS
 Text GLabel 9950 1400 0    60   Input ~ 0
@@
 Text GLabel 9950 1300 0    60   Input ~ 0
 SCREEN_A0
-Text GLabel 1700 6100 0    60   Output ~ 0
+Text GLabel 1700 5900 0    60   Output ~ 0
 SCREEN_A0
 Text GLabel 1700 4900 0    50   Output ~ 0
@@
 Text GLabel 1700 5200 0    50   Output ~ 0
 ~SPI1_CS_3
-Text GLabel 1700 5800 0    50   Output ~ 0
+Text GLabel 7500 5400 2    50   Output ~ 0
 ~SPI1_CS_4
 Text GLabel 7850 1600 0    50   Input ~ 0

Commit message: Adding new FPC-connected board for extra connectors, can transceiver, voltage regulator.
Connections:
- net labels added: ~SPI_CS_5
Changed lines of the file:
@@
 ~ENABLE_SCREEN
 Text GLabel 9950 1200 0    60   Input ~ 0
-~ENABLE_SCREEN
+~SPI_CS_5
 Text GLabel 9950 1500 0    60   Input ~ 0
 ~SCREEN_CS

Commit message: Finishing-up secondary connector board.
Connections:
- net labels added: ~ENABLE_CAN, ~SPI_CS_4
- net labels removed: ~ENABLE_SCREEN_BACKLIGHT, ~SPI1_CS_4, ~SPI_CS_5
Changed lines of the file:
@@
 WAKE
 Text GLabel 7500 6100 2    60   Output ~ 0
-~ENABLE_SCREEN_BACKLIGHT
+~ENABLE_SCREEN
 Text GLabel 7500 5600 2    60   Input ~ 0
 MC_IN
@@
 $EndComp
 Text GLabel 1700 5800 0    60   Output ~ 0
-~ENABLE_SCREEN
+~SPI_CS_4
 Text GLabel 9950 1200 0    60   Input ~ 0
-~SPI_CS_5
+~SPI_CS_4
 Text GLabel 9950 1500 0    60   Input ~ 0
 ~SCREEN_CS
@@
 $EndComp
 Text GLabel 7850 2100 0    60   Input ~ 0
-~ENABLE_SCREEN_BACKLIGHT
+~ENABLE_SCREEN
 Wire Wire Line
 	7550 1200 7550 1300
@@
 ~SPI1_CS_3
 Text GLabel 7500 5400 2    50   Output ~ 0
-~SPI1_CS_4
+~ENABLE_CAN
 Text GLabel 7850 1600 0    50   Input ~ 0
 ~SPI1_CS_2
@@
 ~SPI1_CS_3
 Text GLabel 9950 1600 0    50   Input ~ 0
-~SPI1_CS_4
+~ENABLE_CAN
+Text GLabel 10950 5000 2    60   Input ~ 0
+ESP_BOOT_MODE
 $EndSCHEMATC

Commit message: Updating for manufacture.
Parts:
- U1: footprint kicad-castellated-breakouts:QFP48-1.27MM-CASTELLATED -> kicad-castellated-breakouts:QFP48-1.27MM-CASTELLATED-VERS
Changed lines of the file:
@@
 F 0 "U1" H 4600 6678 50  0000 C CNN
 F 1 "STM32F103C8Tx" H 4600 6587 50  0000 C CNN
-F 2 "kicad-castellated-breakouts:QFP48-1.27MM-CASTELLATED" H 7400 6375 50  0001 R TNN
+F 2 "kicad-castellated-breakouts:QFP48-1.27MM-CASTELLATED-VERS" H 7400 6375 50  0001 R TNN
 F 3 "http://www.st.com/st-web-ui/static/active/en/resource/technical/document/datasheet/CD00161566.pdf" H 4600 4700 50  0001 C CNN
 	1    4600 4700

Commit message: Maxwell Remote v2.0
* Adds WAKE-controlled power switch to save power while sleeping.
* Uses pin headers for connecting upper and lower layers instead
  of FPC connectors.
Parts:
- removed C1, C2, C3, C4: 22p, coddingtonbear/coddingtonbear.pretty:0805_Milling, symbol device:C
- removed C11, C12, C7, C8, C9: 0.1, coddingtonbear/coddingtonbear.pretty:0805_Milling, symbol device:C
- removed J2: UART, coddingtonbear:JST_XH_B03B-XH-A_03x2.50mm_Straight_LargePads, symbol Connector:Conn_01x03
- removed J3: FPC 1, coddingtonbear/coddingtonbear.pretty:10P_FPC_1.0mm, symbol Connector:Conn_01x10
- removed J4: FPC 2, coddingtonbear/coddingtonbear.pretty:10P_FPC_1.0mm, symbol Connector:Conn_01x10
- removed J5: Programmer, coddingtonbear/coddingtonbear.pretty:Pin_Header_Straight_1x04_Pitch2.54mm_LargePads, symbol Connector:Conn_01x04
- removed J6: B0_JMP, coddingtonbear/coddingtonbear.pretty:Pin_Header_Straight_1x02_Pitch1.27mm_JMP, symbol Connector:Conn_01x02
- removed J7: B1_JMP, coddingtonbear/coddingtonbear.pretty:Pin_Header_Straight_1x02_Pitch1.27mm_JMP, symbol Connector:Conn_01x02
- removed J9: ESP_BM, coddingtonbear/coddingtonbear.pretty:Pin_Header_Straight_1x02_Pitch1.27mm_JMP, symbol Connector:Conn_01x02
- removed R1, R5: 100k, coddingtonbear/coddingtonbear.pretty:0805_Milling, symbol device:R
- removed R10: 1M, coddingtonbear/coddingtonbear.pretty:0805_Milling, symbol device:R
- removed R12, R15, R16, R9: 10k, coddingtonbear/coddingtonbear.pretty:0805_Milling, symbol device:R
- removed R7: 330, coddingtonbear/coddingtonbear.pretty:0805_Milling, symbol device:R
- removed U1: STM32F103C8Tx, kicad-castellated-breakouts:QFP48-1.27MM-CASTELLATED-VERS, symbol MCU_ST_STM32:STM32F103C8Tx
- removed U2: ESP32-WROOM, NorbotNorway/NorBotKiCadFootprints.pretty:ESP32-WROOM, symbol esp32-local:ESP32-WROOM
- removed Y1: Crystal, cpavlina/kicad-pcblib/smd-non-ipc.pretty:Abracon-ABM2, symbol device:Crystal
- removed Y2: Crystal_GND23, coddingtonbear:SM-CRYSTAL-ABS25_LargePads, symbol device:Crystal_GND23
- added C1, C2: 22p, coddingtonbear:0805_Milling, symbol Device:C_Small
- added C3, C4, C5, C6, C7: 0.1u, coddingtonbear:0805_Milling, symbol Device:C_Small
- added C8: 220u, coddingtonbear:CP_Tantalum_Case-C_EIA-6032-28_Milling, symbol Device:CP
- added J1: BOOT0, coddingtonbear:Pin_Header_Straight_1x02_Pitch1.27mm_JMP, symbol Connector_Generic:Conn_01x02
- added J2: BOOT1, coddingtonbear:Pin_Header_Straight_1x02_Pitch1.27mm_JMP, symbol Connector_Generic:Conn_01x02
- added J5: Lower-Left, coddingtonbear:PinHeader_2x08_P2.54mm_Vertical_LargePads, symbol Connector_Generic:Conn_02x08_Odd_Even
- added J7: Lower-Right, coddingtonbear:PinHeader_2x08_P2.54mm_Vertical_LargePads, symbol Connector_Generic:Conn_02x08_Odd_Even
- added R1: 1M, coddingtonbear:0805_Milling, symbol Device:R
- added R10, R8, R9: 300, coddingtonbear:0805_Milling, symbol Device:R
- added R2, R7: 10k, coddingtonbear:0805_Milling, symbol Device:R
- added R3, R4: 100k, coddingtonbear:0805_Milling, symbol Device:R
- added U1: STM32F103CBTx, castellated-breakouts:QFP48-1.27MM-CASTELLATED, symbol MCU_ST_STM32F1:STM32F103CBTx
- added U2: ESP32-WROOM-32, RF_Module:ESP32-WROOM-32, symbol RF_Module:ESP32-WROOM-32
- added Y1: 8M, coddingtonbear:Abracon-ABM2_LargePads, symbol Device:Crystal
Connections:
- net labels added: +3V3_A, BT_DI, BT_DO, ESP_AVAILABLE, ESP_DI, ESP_DO, GND_A
- net labels removed: +3V3, BT_IN, BT_OUT, GND, MC_IN, MC_OUT, ~ENABLE_CAN
- wire segments 80 -> 84
- no-connect marks 7 -> 0
