File: hardware/maxwell-remote-2/maxwell-remote-2.sch (KiCad schematic (older format))
At the start: 21 parts, among them J1 INPUT, J2 Left, J3 Right, J4 DISPLAY, J5 FPC-1, J6 FPC-2, J7 SPI1_A, J8 SPI1_B, J9 SPI1_C, Q1 NDS332P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

Commit message: Finishing-up secondary connector board.
Changed lines of the file:
@@
 L power:GND #PWR0101
 U 1 1 5B146099
-P 10050 1050
-F 0 "#PWR0101" H 10050 800 50  0001 C CNN
-F 1 "GND" V 10055 922 50  0000 R CNN
-F 2 "" H 10050 1050 50  0001 C CNN
-F 3 "" H 10050 1050 50  0001 C CNN
-	1    10050 1050
+P 10050 1950
+F 0 "#PWR0101" H 10050 1700 50  0001 C CNN
+F 1 "GND" V 10055 1822 50  0000 R CNN
+F 2 "" H 10050 1950 50  0001 C CNN
+F 3 "" H 10050 1950 50  0001 C CNN
+	1    10050 1950
 	0    1    1    0
 $EndComp
@@
 L power:+3V3 #PWR0102
 U 1 1 5B14611E
-P 10050 1150
-F 0 "#PWR0102" H 10050 1000 50  0001 C CNN
-F 1 "+3V3" V 10065 1278 50  0000 L CNN
-F 2 "" H 10050 1150 50  0001 C CNN
-F 3 "" H 10050 1150 50  0001 C CNN
-	1    10050 1150
+P 10050 1850
+F 0 "#PWR0102" H 10050 1700 50  0001 C CNN
+F 1 "+3V3" V 10065 1978 50  0000 L CNN
+F 2 "" H 10050 1850 50  0001 C CNN
+F 3 "" H 10050 1850 50  0001 C CNN
+	1    10050 1850
 	0    -1   -1   0
 $EndComp
-Text GLabel 10050 1250 0    50   Output ~ 0
+Text GLabel 10050 1750 0    50   Output ~ 0
 CAN_TX
-Text GLabel 10050 1350 0    50   Input ~ 0
+Text GLabel 10050 1650 0    50   Input ~ 0
 CAN_RX
+Text GLabel 10050 1550 0    50   Output ~ 0
+~SPI1_CS_2
 Text GLabel 10050 1450 0    50   Output ~ 0
-~SPI1_CS_2
-Text GLabel 10050 1550 0    50   Output ~ 0
 ~SPI1_CS_3
-Text GLabel 10050 1650 0    50   Output ~ 0
+Text GLabel 10050 1350 0    50   Output ~ 0
 SPI1_MOSI
-Text GLabel 10050 1750 0    50   Input ~ 0
+Text GLabel 10050 1250 0    50   Input ~ 0
 SPI1_MISO
-Text GLabel 10050 1850 0    50   Output ~ 0
+Text GLabel 10050 1150 0    50   Output ~ 0
 SPI1_SCK
+Text GLabel 10050 2800 0    50   Output ~ 0
+~ENABLE_CAN
+Text GLabel 10050 3100 0    50   Output ~ 0
+SCREEN_A0
+Text GLabel 10050 3000 0    50   Output ~ 0
+~SCREEN_RST
+Text GLabel 10050 2900 0    50   Output ~ 0
+~SCREEN_CS
+Text GLabel 10050 3200 0    50   Output ~ 0
+~SPI_CS_4
 Text GLabel 10050 2700 0    50   Output ~ 0
-~ENABLE_CAN
+~RIGHT_B
+Text GLabel 10050 2600 0    50   Output ~ 0
+~RIGHT_A
+Text GLabel 10050 2500 0    50   Output ~ 0
+~LEFT_B
 Text GLabel 10050 2400 0    50   Output ~ 0
-SCREEN_A0
-Text GLabel 10050 2500 0    50   Output ~ 0
-~SCREEN_RST
-Text GLabel 10050 2600 0    50   Output ~ 0
-~SCREEN_CS
-Text GLabel 10050 2300 0    50   Output ~ 0
-~SPI_CS_4
-Text GLabel 10050 2800 0    50   Output ~ 0
-~RIGHT_B
-Text GLabel 10050 2900 0    50   Output ~ 0
-~RIGHT_A
-Text GLabel 10050 3000 0    50   Output ~ 0
-~LEFT_B
-Text GLabel 10050 3100 0    50   Output ~ 0
 ~LEFT_A
-Text GLabel 10050 3200 0    50   BiDi ~ 0
+Text GLabel 10050 2300 0    50   BiDi ~ 0
 WAKE
-Text GLabel 10050 1950 0    50   Output ~ 0
+Text GLabel 10050 1050 0    50   Output ~ 0
 ENABLE_SCREEN
 Text GLabel 5500 850  2    50   Input ~ 0

Commit message: Fixing footprint for MOSFET packages; enable/disable VBATT instead of GND for screen.
Parts:
- Q1: footprint cuzdaori/KiCad.pretty:SOT-23_Handsoldering -> re-innovation/kicad_reinnovation/KiCAD PRETTY/TO_SOT_Packages_SMD.pretty:SOT-23_Handsoldering
- Q2: value BSS138P -> NDS332P; footprint cuzdaori/KiCad.pretty:SOT-23_Handsoldering -> re-innovation/kicad_reinnovation/KiCAD PRETTY/TO_SOT_Packages_SMD.pretty:SOT-23_Handsoldering
Connections:
- wire segments 69 -> 70
Changed lines of the file:
@@
 Text GLabel 10050 1050 0    50   Output ~ 0
 ENABLE_SCREEN
-Text GLabel 5500 850  2    50   Input ~ 0
+Text GLabel 6450 1350 0    50   Input ~ 0
 ENABLE_SCREEN
 $Comp
@@
 L power:+BATT #PWR0103
 U 1 1 5B148AAB
-P 7200 1050
-F 0 "#PWR0103" H 7200 900 50  0001 C CNN
-F 1 "+BATT" H 7215 1223 50  0000 C CNN
-F 2 "" H 7200 1050 50  0001 C CNN
-F 3 "" H 7200 1050 50  0001 C CNN
-	1    7200 1050
+P 5950 1050
+F 0 "#PWR0103" H 5950 900 50  0001 C CNN
+F 1 "+BATT" H 5965 1223 50  0000 C CNN
+F 2 "" H 5950 1050 50  0001 C CNN
+F 3 "" H 5950 1050 50  0001 C CNN
+	1    5950 1050
 	1    0    0    -1
 $EndComp
@@
 F 0 "Q1" V 2193 1250 50  0000 C CNN
 F 1 "NDS332P" V 2102 1250 50  0000 C CNN
-F 2 "cuzdaori/KiCad.pretty:SOT-23_Handsoldering" H 2050 1350 50  0001 C CNN
+F 2 "re-innovation/kicad_reinnovation/KiCAD PRETTY/TO_SOT_Packages_SMD.pretty:SOT-23_Handsoldering" H 2050 1350 50  0001 C CNN
 F 3 "" H 1850 1250 50  0001 C CNN
 	1    1850 1250
@@
 L power:GND #PWR0112
 U 1 1 5B14F63A
-P 5300 1150
-F 0 "#PWR0112" H 5300 900 50  0001 C CNN
-F 1 "GND" V 5305 1022 50  0000 R CNN
-F 2 "" H 5300 1150 50  0001 C CNN
-F 3 "" H 5300 1150 50  0001 C CNN
-	1    5300 1150
-	1    0    0    -1
+P 7200 1150
+F 0 "#PWR0112" H 7200 900 50  0001 C CNN
+F 1 "GND" V 7205 1022 50  0000 R CNN
+F 2 "" H 7200 1150 50  0001 C CNN
+F 3 "" H 7200 1150 50  0001 C CNN
+	1    7200 1150
+	0    1    1    0
 $EndComp
 $Comp
@@
 L device:Q_NMOS_GSD Q2
 U 1 1 5B1502DD
-P 5500 1050
-F 0 "Q2" V 5843 1050 50  0000 C CNN
-F 1 "BSS138P" V 5752 1050 50  0000 C CNN
-F 2 "cuzdaori/KiCad.pretty:SOT-23_Handsoldering" H 5700 1150 50  0001 C CNN
-F 3 "" H 5500 1050 50  0001 C CNN
-	1    5500 1050
-	0    1    1    0
-$EndComp
-Wire Wire Line
-	5700 1150 7200 1150
+P 6450 1150
+F 0 "Q2" V 6793 1150 50  0000 C CNN
+F 1 "NDS332P" V 6702 1150 50  0000 C CNN
+F 2 "re-innovation/kicad_reinnovation/KiCAD PRETTY/TO_SOT_Packages_SMD.pretty:SOT-23_Handsoldering" H 6650 1250 50  0001 C CNN
+F 3 "" H 6450 1150 50  0001 C CNN
+	1    6450 1150
+	0    -1   -1   0
+$EndComp
 $Comp
 L Connector:Conn_01x07 J7
@@
 Text GLabel 1700 2100 0    50   BiDi ~ 0
 CAN+
+Wire Wire Line
+	6650 1050 7200 1050
+Wire Wire Line
+	6250 1050 5950 1050
 $EndSCHEMATC

Commit message: Updating schematics/layouts to latest versions.
Parts:
- C1, C3: symbol device:CP -> maxwell-remote-2-rescue:CP-device
- C2: symbol device:C -> maxwell-remote-2-rescue:C-device
- J1: symbol Connector:Conn_01x05 -> maxwell-remote-2-rescue:Conn_01x05-Connector
- J2, J3: symbol Connector:Conn_01x03 -> maxwell-remote-2-rescue:Conn_01x03-Connector
- J4: symbol Connector:Conn_01x08 -> maxwell-remote-2-rescue:Conn_01x08-Connector
- J5, J6: symbol Connector:Conn_01x10 -> maxwell-remote-2-rescue:Conn_01x10-Connector
- J7, J8, J9: symbol Connector:Conn_01x07 -> maxwell-remote-2-rescue:Conn_01x07-Connector
- Q1: symbol device:Q_PMOS_GSD -> maxwell-remote-2-rescue:Q_PMOS_GSD-device
- Q2: symbol device:Q_NMOS_GSD -> maxwell-remote-2-rescue:Q_NMOS_GSD-device
- R1, R2, R3, R4, R5: symbol device:R -> maxwell-remote-2-rescue:R-device
- U1: symbol interface:SN65HVD235 -> maxwell-remote-2-rescue:SN65HVD235-interface
- U2: symbol coddingtonbear:MIC5209-ADJ -> maxwell-remote-2-rescue:MIC5209-ADJ-coddingtonbear
Changed lines of the file:
@@
 $EndDescr
 $Comp
-L Connector:Conn_01x10 J5
+L maxwell-remote-2-rescue:Conn_01x10-Connector J5
 U 1 1 5B145F18
 P 10250 1450
@@
 $EndComp
 $Comp
-L Connector:Conn_01x10 J6
+L maxwell-remote-2-rescue:Conn_01x10-Connector J6
 U 1 1 5B145F48
 P 10250 2700
@@
 ENABLE_SCREEN
 $Comp
-L Connector:Conn_01x08 J4
+L maxwell-remote-2-rescue:Conn_01x08-Connector J4
 U 1 1 5B148703
 P 7400 1350
@@
 $EndComp
 $Comp
-L Connector:Conn_01x05 J1
+L maxwell-remote-2-rescue:Conn_01x05-Connector J1
 U 1 1 5B148BDD
 P 1250 1250
@@
 $EndComp
 $Comp
-L coddingtonbear:MIC5209-ADJ U2
+L maxwell-remote-2-rescue:MIC5209-ADJ-coddingtonbear U2
 U 1 1 5B148E82
 P 3350 1250
@@
 $EndComp
 $Comp
-L device:R R2
+L maxwell-remote-2-rescue:R-device R2
 U 1 1 5B148F2F
 P 2550 1050
@@
 $EndComp
 $Comp
-L device:Q_PMOS_GSD Q1
+L maxwell-remote-2-rescue:Q_PMOS_GSD-device Q1
 U 1 1 5B148F9A
 P 1850 1250
@@
 $EndComp
 $Comp
-L device:CP C1
+L maxwell-remote-2-rescue:CP-device C1
 U 1 1 5B1491D3
 P 2150 1300
@@
 	2150 1150 2900 1150
 $Comp
-L device:CP C3
+L maxwell-remote-2-rescue:CP-device C3
 U 1 1 5B149293
 P 2550 1400
@@
 Connection ~ 2550 1250
 $Comp
-L device:R R3
+L maxwell-remote-2-rescue:R-device R3
 U 1 1 5B149456
 P 2750 1400
@@
 	2750 1250 2550 1250
 $Comp
-L device:R R4
+L maxwell-remote-2-rescue:R-device R4
 U 1 1 5B149498
 P 2750 1750
@@
 Connection ~ 3800 1350
 $Comp
-L interface:SN65HVD235 U1
+L maxwell-remote-2-rescue:SN65HVD235-interface U1
 U 1 1 5B14A98D
 P 2350 3050
@@
 $EndComp
 $Comp
-L device:C C2
+L maxwell-remote-2-rescue:C-device C2
 U 1 1 5B14AA77
 P 2200 3500
@@
 ~ENABLE_CAN
 $Comp
-L device:R R5
+L maxwell-remote-2-rescue:R-device R5
 U 1 1 5B14C80B
 P 2800 2700
@@
 Connection ~ 2800 2850
 $Comp
-L device:R R1
+L maxwell-remote-2-rescue:R-device R1
 U 1 1 5B14E249
 P 1500 2600
@@
 SPI1_MOSI
 $Comp
-L Connector:Conn_01x03 J2
+L maxwell-remote-2-rescue:Conn_01x03-Connector J2
 U 1 1 5B14FA4E
 P 5300 2700
@@
 $EndComp
 $Comp
-L Connector:Conn_01x03 J3
+L maxwell-remote-2-rescue:Conn_01x03-Connector J3
 U 1 1 5B14FAD5
 P 6750 2700
@@
 ~RIGHT_B
 $Comp
-L device:Q_NMOS_GSD Q2
+L maxwell-remote-2-rescue:Q_NMOS_GSD-device Q2
 U 1 1 5B1502DD
 P 6450 1150
@@
 $EndComp
 $Comp
-L Connector:Conn_01x07 J7
+L maxwell-remote-2-rescue:Conn_01x07-Connector J7
 U 1 1 5B152945
 P 7950 3400
@@
 $EndComp
 $Comp
-L Connector:Conn_01x07 J8
+L maxwell-remote-2-rescue:Conn_01x07-Connector J8
 U 1 1 5B1529E8
 P 7950 3850
@@
 $EndComp
 $Comp
-L Connector:Conn_01x07 J9
+L maxwell-remote-2-rescue:Conn_01x07-Connector J9
 U 1 1 5B152A24
 P 7950 4350
